File: Kicad_dev/Kicad_dev.kicad_sch (KiCad schematic)
At the start: 33 parts, among them J1 Conn_01x02_Pin, J2 Conn_01x02_Pin, J3 Conn_01x02_Pin, J4 530470510_Picoblade, J5 Connecteur_SMA, J6 BNC, Q1 IRF540N, SW1 RotaryEncoder_Switch, SW2 RotaryEncoder_Switch, U11 MAX-8Q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

Commit message: Add repo of lib Kicad before analyzing...
Parts:
- added U1: COM-09032, CREPP_Joysticks:XDCR_COM-09032_V2, symbol CREPP_Joysticks:COM-09032_JOYSTICK
- OLED1: footprint CREPP_Screens:SSD1306_OLED_Display(128x64) -> CREPP_Screens:SSD1306_OLED_Display_128_64_VIRTUAL
Connections:
- new net: U1.S1 (SHIELD), U1.S2 (SHIELD), U1.S3 (SHIELD), U1.S4 (SHIELD)
Changed lines of the file:
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@@
 			)
 		)
-		(property "Footprint" "CREPP_Screens:SSD1306_OLED_Display(128x64)"
+		(property "Footprint" "CREPP_Screens:SSD1306_OLED_Display_128_64_VIRTUAL"
 			(at 78.74 44.45 0)
 			(effects
@@
 					(unit 1)
 				)
+			)
+		)
+	)
+	(symbol
+		(lib_id "CREPP_Joysticks:COM-09032_JOYSTICK")
+		(at 41.91 76.2 0)
+		(unit 1)
+		(exclude_from_sim no)
+		(in_bom yes)
+		(on_board yes)
+		(dnp no)
+		(fields_autoplaced yes)
+		(property "Reference" "U1"
+			(at 50.8 76.1999 0)
+			(effects
+				(font
+					(size 1.27 1.27)
+				)
+				(justify left)
+			)
+		)
+		(property "Value" "COM-09032"
+			(at 50.8 78.7399 0)
+			(effects
+				(font
+					(size 1.27 1.27)
+				)
+				(justify left)
+			)
+		)
+		(property "Footprint" "CREPP_Joysticks:XDCR_COM-09032_V2"
+			(at 41.91 76.2 0)
+			(effects
+				(font
+					(size 1.27 1.27)
+				)
+				(justify bottom)
+				(hide yes)
+			)
+		)
+		(property "Datasheet" ""
+			(at 41.91 76.2 0)
+			(effects
+				(font
+					(size 1.27 1.27)
+				)
+				(hide yes)
+			)
+		)
+		(property "Description" ""
+			(at 41.91 76.2 0)
+			(effects
+				(font
+					(size 1.27 1.27)
+				)
+				(hide yes)
+			)
+		)
+		(property "MF" "SparkFun Electronics"
+			(at 41.91 76.2 0)
+			(effects
+				(font
+					(size 1.27 1.27)
+				)
+				(justify bottom)
+				(hide yes)
+			)
+		)
+		(property "MAXIMUM_PACKAGE_HEIGHT" "30.1mm"
+			(at 41.91 76.2 0)
+			(effects
+				(font
+					(size 1.27 1.27)
+				)
+				(justify bottom)
+				(hide yes)
+			)
+		)
+		(property "Package" "Package"
+			(at 41.91 76.2 0)
+			(effects
+				(font
+					(size 1.27 1.27)
+				)
+				(justify bottom)
+				(hide yes)
+			)
+		)
+		(property "Price" "None"
+			(at 41.91 76.2 0)
+			(effects
+				(font
+					(size 1.27 1.27)
+				)
+				(justify bottom)
+				(hide yes)
+			)
+		)
+		(property "Check_prices" "https://www.snapeda.com/parts/COM-09032/SparkFun/view-part/?ref=eda"
+			(at 41.91 76.2 0)
+			(effects
+				(font
+					(size 1.27 1.27)
+				)
+				(justify bottom)
+				(hide yes)
+			)
+		)
+		(property "STANDARD" "Manufacturer Recommendations"
+			(at 41.91 76.2 0)
+			(effects
+				(font
+					(size 1.27 1.27)
+				)
+				(justify bottom)
+				(hide yes)
+			)
+		)
+		(property "PARTREV" "N/A"
+			(at 41.91 76.2 0)
+			(effects
+				(font
+					(size 1.27 1.27)
+				)
+				(justify bottom)
+				(hide yes)
+			)
+		)
+		(property "SnapEDA_Link" "https://www.snapeda.com/parts/COM-09032/SparkFun/view-part/?ref=snap"
+			(at 41.91 76.2 0)
+			(effects
+				(font
+					(size 1.27 1.27)
+				)
+				(justify bottom)
+				(hide yes)
+			)
+		)
+		(property "MP" "COM-09032"
+			(at 41.91 76.2 0)
+			(effects
+				(font
+					(size 1.27 1.27)
+				)
+				(justify bottom)
+				(hide yes)
+			)
+		)
+		(property "Description_1" "\n                        \n                            Joystick, 2 - Axis Analog (Resistive) Output\n                        \n"
+			(at 41.91 76.2 0)
+			(effects
+				(font
+					(size 1.27 1.27)
+				)
+				(justify bottom)
+				(hide yes)
+			)
+		)
+		(property "Availability" "In Stock"
+			(at 41.91 76.2 0)
+			(effects
+				(font
+					(size 1.27 1.27)
+				)
+				(justify bottom)
+				(hide yes)
+			)
+		)
+		(property "MANUFACTURER" "SparkFun Electronics"
+			(at 41.91 76.2 0)
+			(effects
+				(font
+					(size 1.27 1.27)
+				)
+				(justify bottom)
+				(hide yes)
+			)
+		)
+		(pin "V3"
+		)
+		(pin "S4"
+		)
+		(pin "V1"
+		)
+		(pin "H3"
+		)
+		(pin "V2"
+		)
+		(pin "H2"
+		)
+		(pin "H1"
+		)
+		(pin "B2A"
+		)
+		(pin "S1"
+		)
+		(pin "S3"
+		)
+		(pin "S2"
+		)
+		(pin "B1A"
+		)
+		(instances
+			(project "Kicad_dev"
+				(path "/8104dfe2-da9a-40cd-b518-c622bfb26061"
+					(reference "U1")
+					(unit 1)
+				)

Commit message: Add repo of lib Kicad before analyzing...
Parts:
- OLED1: footprint CREPP_Screens:SSD1306_OLED_Display_128_64_VIRTUAL -> CREPP_Screens:SSD1306_OLED_Display_VIRTUAL_128_64

Commit message: Add repo of lib Kicad before analyzing...
Parts:
- removed U12, U2: COM-09032, CREPP_Joysticks:XDCR_COM-09032, symbol CREPP_Joysticks:COM-09032
- U1: footprint CREPP_Joysticks:XDCR_COM-09032_V2 -> CREPP_Joysticks_SW:XDCR_COM-09032

Commit message: Add repo of lib Kicad before analyzing...
Parts:
- added D1: LED_5mm_THT, LED_SMD:LED_0603_1608Metric, symbol CREPP_LED:LED_0603_CMS
- added D2: LED_5mm_THT, LED_THT:LED_D5.0mm, symbol CREPP_LED:LED_5mm_THT
- added D3: LED_5mm_THT, LED_SMD:LED_0805_2012Metric, symbol CREPP_LED:LED_0805_CMS
Changed lines of the file:
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@@
+	)
+	(symbol
+		(lib_id "CREPP_LED:LED_0805_CMS")
+		(at 273.05 149.86 0)
+		(unit 1)
+		(exclude_from_sim no)
+		(in_bom yes)
+		(on_board yes)
+		(dnp no)
+		(fields_autoplaced yes)
+		(property "Reference" "D3"
+			(at 271.4625 143.51 0)
+			(effects
+				(font
+					(size 1.27 1.27)
+				)
+			)
+		)
+		(property "Value" "LED_5mm_THT"
+			(at 271.4625 146.05 0)
+			(effects
+				(font
+					(size 1.27 1.27)
+				)
+			)
+		)
+		(property "Footprint" "LED_SMD:LED_0805_2012Metric"
+			(at 273.05 149.86 0)
+			(effects
+				(font
+					(size 1.27 1.27)
+				)
+				(hide yes)
+			)
+		)
+		(property "Datasheet" "~"
+			(at 273.05 149.86 0)
+			(effects
+				(font
+					(size 1.27 1.27)
+				)
+				(hide yes)
+			)
+		)
+		(property "Description" "Light emitting diode"
+			(at 273.05 149.86 0)
+			(effects
+				(font
+					(size 1.27 1.27)
+				)
+				(hide yes)
+			)
+		)
+		(pin "2"
+		)
+		(pin "1"
+		)
+		(instances
+			(project "Kicad_dev"
+				(path "/8104dfe2-da9a-40cd-b518-c622bfb26061"
+					(reference "D3")
+					(unit 1)
+				)
+			)
+		)
 	)
 	(symbol
@@
 	)
 	(symbol
+		(lib_id "CREPP_LED:LED_5mm_THT")
+		(at 273.05 138.43 0)
+		(unit 1)
+		(exclude_from_sim no)
+		(in_bom yes)
+		(on_board yes)
+		(dnp no)
+		(fields_autoplaced yes)
+		(property "Reference" "D2"
+			(at 271.4625 132.08 0)
+			(effects
+				(font
+					(size 1.27 1.27)
+				)
+			)
+		)
+		(property "Value" "LED_5mm_THT"
+			(at 271.4625 134.62 0)
+			(effects
+				(font
+					(size 1.27 1.27)
+				)
+			)
+		)
+		(property "Footprint" "LED_THT:LED_D5.0mm"
+			(at 273.05 138.43 0)
+			(effects
+				(font
+					(size 1.27 1.27)
+				)
+				(hide yes)
+			)
+		)
+		(property "Datasheet" "~"
+			(at 273.05 138.43 0)
+			(effects
+				(font
+					(size 1.27 1.27)
+				)
+				(hide yes)
+			)
+		)
+		(property "Description" "Light emitting diode"
+			(at 273.05 138.43 0)
+			(effects
+				(font
+					(size 1.27 1.27)
+				)
+				(hide yes)
+			)
+		)
+		(pin "1"
+		)
+		(pin "2"
+		)
+		(instances
+			(project "Kicad_dev"
+				(path "/8104dfe2-da9a-40cd-b518-c622bfb26061"
+					(reference "D2")
+					(unit 1)
+				)
+			)
+		)
+	)
+	(symbol
 		(lib_id "CREPP_Heatsinks:Heatsink")
 		(at 105.41 110.49 0)
@@
 					(unit 1)
 				)
+			)
+		)
+	)
+	(symbol
+		(lib_id "CREPP_LED:LED_0603_CMS")
+		(at 273.05 125.73 0)
+		(unit 1)
+		(exclude_from_sim no)
+		(in_bom yes)
+		(on_board yes)
+		(dnp no)
+		(fields_autoplaced yes)
+		(property "Reference" "D1"
+			(at 271.4625 119.38 0)
+			(effects
+				(font
+					(size 1.27 1.27)
+				)
+			)
+		)
+		(property "Value" "LED_5mm_THT"
+			(at 271.4625 121.92 0)
+			(effects
+				(font
+					(size 1.27 1.27)
+				)
+			)
+		)
+		(property "Footprint" "LED_SMD:LED_0603_1608Metric"
+			(at 273.05 125.73 0)
+			(effects
+				(font
+					(size 1.27 1.27)
+				)
+				(hide yes)
+			)
+		)
+		(property "Datasheet" "~"
+			(at 273.05 125.73 0)
+			(effects
+				(font
+					(size 1.27 1.27)
+				)
+				(hide yes)
+			)
+		)
+		(property "Description" "Light emitting diode"
+			(at 273.05 125.73 0)
+			(effects
+				(font
+					(size 1.27 1.27)
+				)
+				(hide yes)
+			)
+		)
+		(pin "2"
+		)
+		(pin "1"
+		)
+		(instances
+			(project "Kicad_dev"
+				(path "/8104dfe2-da9a-40cd-b518-c622bfb26061"
+					(reference "D1")
+					(unit 1)
+				)

Commit message: Add repo of lib Kicad before analyzing...
Parts:
- added C1, C2: Supercapacitors_D10mm_H20mm, CREPP_Capacitors_THT:C_Radial_D10.0mm_H20.0mm_P5.00mm, symbol CREPP_Capacitors_THT:Supercapacitors_D10mm_H20mm
- added R3: R_0805, Resistor_SMD:R_0805_2012Metric, symbol CREPP_Resistors:R_0805
- added U12: LM317_TO-220, Package_TO_SOT_THT:TO-220-3_Vertical, symbol CREPP_Voltage_regulators_THT:LM317_TO-220
- added U13: LM7805_TO220, Package_TO_SOT_THT:TO-220-3_Vertical, symbol CREPP_Voltage_regulators_THT:LM7805_TO220
- added U2: LM317_SOT-223, Package_TO_SOT_SMD:SOT-223-3_TabPin2, symbol CREPP_Voltage_regulators_SMT:LM317_SOT-223

Commit message: Add repo of lib Kicad before analyzing...
Parts:
- added D4: SS24, Diode_SMD:D_SMA, symbol CREPP_Diodes_SMT:SS24
- added RV1: R_Potentiometer, Potentiometer_THT:Potentiometer_Alps_RK163_Single_Horizontal, symbol CREPP_Potentiometers_THT:R_Potentiometer
Changed lines of the file:
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@@
+	)
+	(symbol
+		(lib_id "CREPP_Diodes_SMT:SS24")
+		(at 134.62 130.81 0)
+		(unit 1)
+		(exclude_from_sim no)
+		(in_bom yes)
+		(on_board yes)
+		(dnp no)
+		(fields_autoplaced yes)
+		(property "Reference" "D4"
+			(at 134.3025 124.46 0)
+			(effects
+				(font
+					(size 1.27 1.27)
+				)
+			)
+		)
+		(property "Value" "SS24"
+			(at 134.3025 127 0)
+			(effects
+				(font
+					(size 1.27 1.27)
+				)
+			)
+		)
+		(property "Footprint" "Diode_SMD:D_SMA"
+			(at 134.62 135.255 0)
+			(effects
+				(font
+					(size 1.27 1.27)
+				)
+				(hide yes)
+			)
+		)
+		(property "Datasheet" "https://www.vishay.com/docs/88748/ss22.pdf"
+			(at 134.62 130.81 0)
+			(effects
+				(font
+					(size 1.27 1.27)
+				)
+				(hide yes)
+			)
+		)
+		(property "Description" "40V 2A Schottky Diode, SMA"
+			(at 134.62 130.81 0)
+			(effects
+				(font
+					(size 1.27 1.27)
+				)
+				(hide yes)
+			)
+		)
+		(pin "1"
+		)
+		(pin "2"
+		)
+		(instances
+			(project "Kicad_dev"
+				(path "/8104dfe2-da9a-40cd-b518-c622bfb26061"
+					(reference "D4")
+					(unit 1)
+				)
+			)
+		)
 	)
 	(symbol
@@
 					(unit 1)
 				)
+			)
+		)
+	)
+	(symbol
+		(lib_id "CREPP_Potentiometers_THT:R_Potentiometer")
+		(at 124.46 123.19 0)
+		(unit 1)
+		(exclude_from_sim no)
+		(in_bom yes)
+		(on_board yes)
+		(dnp no)
+		(fields_autoplaced yes)
+		(property "Reference" "RV1"
+			(at 121.92 121.9199 0)
+			(effects
+				(font
+					(size 1.27 1.27)
+				)
+				(justify right)
+			)
+		)
+		(property "Value" "R_Potentiometer"
+			(at 121.92 124.4599 0)
+			(effects
+				(font
+					(size 1.27 1.27)
+				)
+				(justify right)
+			)
+		)
+		(property "Footprint" "Potentiometer_THT:Potentiometer_Alps_RK163_Single_Horizontal"
+			(at 124.46 123.19 0)
+			(effects
+				(font
+					(size 1.27 1.27)
+				)
+				(hide yes)
+			)
+		)
+		(property "Datasheet" "~"
+			(at 124.46 123.19 0)
+			(effects
+				(font
+					(size 1.27 1.27)
+				)
+				(hide yes)
+			)
+		)
+		(property "Description" "Potentiometer"
+			(at 124.46 123.19 0)
+			(effects
+				(font
+					(size 1.27 1.27)
+				)
+				(hide yes)
+			)
+		)
+		(pin "2"
+		)
+		(pin "1"
+		)
+		(pin "3"
+		)
+		(instances
+			(project "Kicad_dev"
+				(path "/8104dfe2-da9a-40cd-b518-c622bfb26061"
+					(reference "RV1")
+					(unit 1)
+				)

Commit message: Add repo of lib Kicad before analyzing...
Parts:
- added R4: LDR03, OptoDevice:R_LDR_7x6mm_P5.1mm_Vertical, symbol CREPP_Light_sensors:LDR03
- added U14: DHT11, Sensor:Aosong_DHT11_5.5x12.0_P2.54mm, symbol CREPP_Temperature_sensors:DHT11
- added U15: DHT11, Sensor:Aosong_DHT11_5.5x12.0_P2.54mm, symbol CREPP_Temperature_sensors:DHT22
- added U16: ~, symbol CREPP_Temperature_sensors:BME280_Breakout

Commit message: Add repo of lib Kicad before analyzing...
Parts:
- added SW3: SW_DPST_x2, Button_Switch_SMD:SW_SPST_PTS645, symbol CREPP_Buttons_SMT:SW_DPST_x2
- added SW4: SW_DPST_x2, Button_Switch_THT:SW_PUSH_6mm_H4.3mm, symbol CREPP_Buttons_THT:SW_DPST_x2
- added U17: ATmega328-A, Package_QFP:TQFP-32_7x7mm_P0.8mm, symbol CREPP_MCU_ATMEL:ATmega328-A
- added U18: ATmega328-P, Package_DIP:DIP-28_W7.62mm, symbol CREPP_MCU_ATMEL:ATmega328-P
- added U19: STM32F030CCTx, Package_QFP:LQFP-48_7x7mm_P0.5mm, symbol CREPP_MCU_STM32:STM32F030CCTx
- added U20: STM32F446VETx, Package_QFP:LQFP-100_14x14mm_P0.5mm, symbol CREPP_MCU_STM32:STM32F446VETx
- added U21: STM32F723ZETx, Package_QFP:LQFP-144_20x20mm_P0.5mm, symbol CREPP_MCU_STM32:STM32F723ZETx
- added U22: MPU-6050, Sensor_Motion:InvenSense_QFN-24_4x4mm_P0.5mm, symbol CREPP_Accelerometers:MPU-6050
Connections:
- new net: U19.23 (VSS), U19.35 (VSS), U19.47 (VSS)
- new net: U17.21 (GND), U17.3 (GND), U17.5 (GND)
- new net: U17.4 (VCC), U17.6 (VCC)
- new net: U21.107 (VSS), U21.120 (VSS), U21.130 (VSS), U21.16 (VSS), U21.38 (VSS), U21.51 (VSS), U21.61 (VSS), U21.85 (VSS), U21.94 (VSS)
- new net: U18.22 (GND), U18.8 (GND)
- new net: U20.10 (VSS), U20.27 (VSS), U20.49 (VSS), U20.74 (VSS), U20.99 (VSS)
