File: Kicad_dev/Kicad_dev.kicad_sch (KiCad schematic)
At the start: 55 parts, among them J1 Conn_01x02_Pin, J2 Conn_01x02_Pin, J3 Conn_01x02_Pin, J4 530470510_Picoblade, J5 Connecteur_SMA, J6 BNC, Q1 IRF540N, SW1 RotaryEncoder_Switch, SW2 RotaryEncoder_Switch, SW3 SW_DPST_x2, SW4 SW_DPST_x2, U1 COM-09032, U11 MAX-8Q, U12 LM317_TO-220, U13 LM7805_TO220, U14 DHT11, U15 DHT11, U17 ATmega328-A, U18 ATmega328-P, U19 STM32F030CCTx, U2 LM317_SOT-223, U20 STM32F446VETx, U21 STM32F723ZETx, U22 MPU-6050, U3 74HC04, U4 L293D, U5 LM358, U6 PC817_SMD, U7 PC817_THT, U8 NEO-M8Q

Commit message: Add repo of lib Kicad before analyzing...
Parts:
- added BT1: Battery_Cell, BC501SM:MPD_BC501SM-TR, symbol CREPP_Batteries:Battery_Cell
- added U23: DS1307+, Package_DIP:DIP-8_W7.62mm_Socket, symbol CREPP_RTC:DS1307+
- added U24: DS3231M, Package_SO:SOIC-16W_7.5x10.3mm_P1.27mm, symbol CREPP_RTC:DS3231M
Connections:
- new net: U24.10 (GND), U24.11 (GND), U24.12 (GND), U24.13 (GND), U24.5 (GND), U24.6 (GND), U24.7 (GND), U24.8 (GND), U24.9 (GND)
Changed lines of the file:
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@@
 	)
 	(symbol
+		(lib_id "CREPP_Batteries:Battery_Cell")
+		(at 149.86 58.42 0)
+		(unit 1)
+		(exclude_from_sim no)
+		(in_bom yes)
+		(on_board yes)
+		(dnp no)
+		(fields_autoplaced yes)
+		(property "Reference" "BT1"
+			(at 153.67 55.3084 0)
+			(effects
+				(font
+					(size 1.27 1.27)
+				)
+				(justify left)
+			)
+		)
+		(property "Value" "Battery_Cell"
+			(at 153.67 57.8484 0)
+			(effects
+				(font
+					(size 1.27 1.27)
+				)
+				(justify left)
+			)
+		)
+		(property "Footprint" "BC501SM:MPD_BC501SM-TR"
+			(at 149.86 56.896 90)
+			(effects
+				(font
+					(size 1.27 1.27)
+				)
+				(hide yes)
+			)
+		)
+		(property "Datasheet" "~"
+			(at 149.86 56.896 90)
+			(effects
+				(font
+					(size 1.27 1.27)
+				)
+				(hide yes)
+			)
+		)
+		(property "Description" "Single-cell battery"
+			(at 149.86 58.42 0)
+			(effects
+				(font
+					(size 1.27 1.27)
+				)
+				(hide yes)
+			)
+		)
+		(pin "2"
+		)
+		(pin "1"
+		)
+		(instances
+			(project "Kicad_dev"
+				(path "/8104dfe2-da9a-40cd-b518-c622bfb26061"
+					(reference "BT1")
+					(unit 1)
+				)
+			)
+		)
+	)
+	(symbol
 		(lib_id "CREPP_Optocoupler:PC817_SMD")
 		(at 27.94 170.18 0)
@@
 	)
 	(symbol
+		(lib_id "CREPP_RTC:DS3231M")
+		(at 69.85 -22.86 0)
+		(unit 1)
+		(exclude_from_sim no)
+		(in_bom yes)
+		(on_board yes)
+		(dnp no)
+		(fields_autoplaced yes)
+		(property "Reference" "U24"
+			(at 72.0441 -11.43 0)
+			(effects
+				(font
+					(size 1.27 1.27)
+				)
+				(justify left)
+			)
+		)
+		(property "Value" "DS3231M"
+			(at 72.0441 -8.89 0)
+			(effects
+				(font
+					(size 1.27 1.27)
+				)
+				(justify left)
+			)
+		)
+		(property "Footprint" "Package_SO:SOIC-16W_7.5x10.3mm_P1.27mm"
+			(at 69.85 -7.62 0)
+			(effects
+				(font
+					(size 1.27 1.27)
+				)
+				(hide yes)
+			)
+		)
+		(property "Datasheet" "http://datasheets.maximintegrated.com/en/ds/DS3231.pdf"
+			(at 76.708 -24.13 0)
+			(effects
+				(font
+					(size 1.27 1.27)
+				)
+				(hide yes)
+			)
+		)
+		(property "Description" "Extremely Accurate I2C-Integrated RTC/TCXO/Crystal SOIC-16"
+			(at 69.85 -22.86 0)
+			(effects
+				(font
+					(size 1.27 1.27)
+				)
+				(hide yes)
+			)
+		)
+		(pin "1"
+		)
+		(pin "12"
+		)
+		(pin "15"
+		)
+		(pin "5"
+		)
+		(pin "14"
+		)
+		(pin "4"
+		)
+		(pin "13"
+		)
+		(pin "7"
+		)
+		(pin "16"
+		)
+		(pin "9"
+		)
+		(pin "11"
+		)
+		(pin "10"
+		)
+		(pin "6"
+		)
+		(pin "2"
+		)
+		(pin "8"
+		)
+		(pin "3"
+		)
+		(instances
+			(project "Kicad_dev"
+				(path "/8104dfe2-da9a-40cd-b518-c622bfb26061"
+					(reference "U24")
+					(unit 1)
+				)
+			)
+		)
+	)
+	(symbol
 		(lib_id "CREPP_Connectors_SMA:Connecteur_SMA")
 		(at 90.17 170.18 0)
@@
 					(unit 1)
 				)
+			)
+		)
+	)
+	(symbol
+		(lib_id "CREPP_RTC:DS1307+")
+		(at 104.14 -22.86 0)
+		(unit 1)
+		(exclude_from_sim no)
+		(in_bom yes)
+		(on_board yes)
+		(dnp no)
+		(fields_autoplaced yes)
+		(property "Reference" "U23"
+			(at 120.65 -29.1786 0)
+			(effects
+				(font
+					(size 1.27 1.27)
+				)
+			)
+		)
+		(property "Value" "DS1307+"
+			(at 120.65 -26.6386 0)
+			(effects
+				(font
+					(size 1.27 1.27)
+				)
+			)
+		)
+		(property "Footprint" "Package_DIP:DIP-8_W7.62mm_Socket"
+			(at 104.14 -10.16 0)
+			(effects
+				(font
+					(size 1.27 1.27)
+				)
+				(hide yes)
+			)
+		)
+		(property "Datasheet" "https://datasheets.maximintegrated.com/en/ds/DS1307.pdf"
+			(at 104.14 -17.78 0)
+			(effects
+				(font
+					(size 1.27 1.27)
+				)
+				(hide yes)
+			)
+		)
+		(property "Description" "64 x 8, Serial, I2C Real-time clock, 4.5V to 5.5V VCC, 0°C to +70°C, DIP-8"
+			(at 104.14 -22.86 0)
+			(effects
+				(font
+					(size 1.27 1.27)
+				)
+				(hide yes)
+			)
+		)
+		(pin "8"
+		)
+		(pin "5"
+		)
+		(pin "2"
+		)
+		(pin "1"
+		)
+		(pin "6"
+		)
+		(pin "4"
+		)
+		(pin "3"
+		)
+		(pin "7"
+		)
+		(instances
+			(project "Kicad_dev"
+				(path "/8104dfe2-da9a-40cd-b518-c622bfb26061"
+					(reference "U23")
+					(unit 1)
+				)

Commit message: Add repo of lib Kicad before analyzing...
Parts:
- removed U9: ~, symbol CREPP_Batteries:BK-18650-PC2_18650_Holder_THT [CREPP]
- added U25: ~, CREPP_Battery_Holders:BK-18650-PC2_18650_Holder_THT [CREPP], symbol CREPP_Batteries:BK-18650-PC2_18650_Holder_THT [CREPP]
Changed lines of the file:
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@@
 	)
 	(symbol
+		(lib_name "BK-18650-PC2_18650_Holder_THT [CREPP]_1")
+		(lib_id "CREPP_Batteries:BK-18650-PC2_18650_Holder_THT [CREPP]")
+		(at 77.47 101.6 0)
+		(unit 1)
+		(exclude_from_sim no)
+		(in_bom yes)
+		(on_board yes)
+		(dnp no)
+		(fields_autoplaced yes)
+		(property "Reference" "U25"
+			(at 80.01 104.1399 0)
+			(effects
+				(font
+					(size 1.27 1.27)
+				)
+				(justify left)
+			)
+		)
+		(property "Value" "~"
+			(at 80.01 106.045 0)
+			(effects
+				(font
+					(size 1.27 1.27)
+				)
+				(justify left)
+			)
+		)
+		(property "Footprint" "CREPP_Battery_Holders:BK-18650-PC2_18650_Holder_THT [CREPP]"
+			(at 77.47 101.6 0)
+			(effects
+				(font
+					(size 1.27 1.27)
+				)
+				(hide yes)
+			)
+		)
+		(property "Datasheet" ""
+			(at 77.47 101.6 0)
+			(effects
+				(font
+					(size 1.27 1.27)
+				)
+				(hide yes)
+			)
+		)
+		(property "Description" ""
+			(at 77.47 101.6 0)
+			(effects
+				(font
+					(size 1.27 1.27)
+				)
+				(hide yes)
+			)
+		)
+		(pin "1"
+		)
+		(pin "1"
+		)
+		(instances
+			(project "Kicad_dev"
+				(path "/8104dfe2-da9a-40cd-b518-c622bfb26061"
+					(reference "U25")
+					(unit 1)
+				)
+			)
+		)
+	)
+	(symbol
 		(lib_id "CREPP_Light_sensors:LDR03")
 		(at 195.58 148.59 0)
@@
 					(unit 1)
 				)
-			)
-		)
-	)
-	(symbol
-		(lib_id "CREPP_Batteries:BK-18650-PC2_18650_Holder_THT [CREPP]")
-		(at 27.94 118.11 0)
-		(unit 1)
-		(exclude_from_sim no)
-		(in_bom yes)
-		(on_board yes)
-		(dnp no)
-		(fields_autoplaced yes)
-		(property "Reference" "U9"
-			(at 30.48 120.6499 0)
-			(effects
-				(font
-					(size 1.27 1.27)
-				)
-				(justify left)
-			)
-		)
-		(property "Value" "~"
-			(at 30.48 122.555 0)
-			(effects
-				(font
-					(size 1.27 1.27)
-				)
-				(justify left)
-			)
-		)
-		(property "Footprint" ""
-			(at 27.94 118.11 0)
-			(effects
-				(font
-					(size 1.27 1.27)
-				)
-				(hide yes)
-			)
-		)
-		(property "Datasheet" ""
-			(at 27.94 118.11 0)
-			(effects
-				(font
-					(size 1.27 1.27)
-				)
-				(hide yes)
-			)
-		)
-		(property "Description" ""
-			(at 27.94 118.11 0)
-			(effects
-				(font
-					(size 1.27 1.27)
-				)
-				(hide yes)
-			)
-		)
-		(pin "1"
-		)
-		(pin "1"
-		)
-		(instances
-			(project "Kicad_dev"
-				(path "/8104dfe2-da9a-40cd-b518-c622bfb26061"
-					(reference "U9")
-					(unit 1)
-				)

Commit message: Add repo of lib Kicad before analyzing...
Parts:
- removed U25: ~, CREPP_Battery_Holders:BK-18650-PC2_18650_Holder_THT [CREPP], symbol CREPP_Batteries:BK-18650-PC2_18650_Holder_THT [CREPP]
- added U9: ~, CREPP_Battery_Holders:BK-18650-PC2_18650_Holder_THT [CREPP], symbol CREPP_Batteries:BK-18650-PC2_18650_Holder_THT [CREPP]
Changed lines of the file:
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@@
-	)
-	(symbol
-		(lib_name "BK-18650-PC2_18650_Holder_THT [CREPP]_1")
-		(lib_id "CREPP_Batteries:BK-18650-PC2_18650_Holder_THT [CREPP]")
-		(at 77.47 101.6 0)
-		(unit 1)
-		(exclude_from_sim no)
-		(in_bom yes)
-		(on_board yes)
-		(dnp no)
-		(fields_autoplaced yes)
-		(property "Reference" "U25"
-			(at 80.01 104.1399 0)
-			(effects
-				(font
-					(size 1.27 1.27)
-				)
-				(justify left)
-			)
-		)
-		(property "Value" "~"
-			(at 80.01 106.045 0)
-			(effects
-				(font
-					(size 1.27 1.27)
-				)
-				(justify left)
-			)
-		)
-		(property "Footprint" "CREPP_Battery_Holders:BK-18650-PC2_18650_Holder_THT [CREPP]"
-			(at 77.47 101.6 0)
-			(effects
-				(font
-					(size 1.27 1.27)
-				)
-				(hide yes)
-			)
-		)
-		(property "Datasheet" ""
-			(at 77.47 101.6 0)
-			(effects
-				(font
-					(size 1.27 1.27)
-				)
-				(hide yes)
-			)
-		)
-		(property "Description" ""
-			(at 77.47 101.6 0)
-			(effects
-				(font
-					(size 1.27 1.27)
-				)
-				(hide yes)
-			)
-		)
-		(pin "1"
-		)
-		(pin "1"
-		)
-		(instances
-			(project "Kicad_dev"
-				(path "/8104dfe2-da9a-40cd-b518-c622bfb26061"
-					(reference "U25")
-					(unit 1)
-				)
-			)
-		)
 	)
 	(symbol
@@
 					(unit 1)
 				)
+			)
+		)
+	)
+	(symbol
+		(lib_id "CREPP_Batteries:BK-18650-PC2_18650_Holder_THT [CREPP]")
+		(at 74.93 105.41 0)
+		(unit 1)
+		(exclude_from_sim no)
+		(in_bom yes)
+		(on_board yes)
+		(dnp no)
+		(fields_autoplaced yes)
+		(property "Reference" "U9"
+			(at 77.47 107.9499 0)
+			(effects
+				(font
+					(size 1.27 1.27)
+				)
+				(justify left)
+			)
+		)
+		(property "Value" "~"
+			(at 77.47 109.855 0)
+			(effects
+				(font
+					(size 1.27 1.27)
+				)
+				(justify left)
+			)
+		)
+		(property "Footprint" "CREPP_Battery_Holders:BK-18650-PC2_18650_Holder_THT [CREPP]"
+			(at 74.93 105.41 0)
+			(effects
+				(font
+					(size 1.27 1.27)
+				)
+				(hide yes)
+			)
+		)
+		(property "Datasheet" ""
+			(at 74.93 105.41 0)
+			(effects
+				(font
+					(size 1.27 1.27)
+				)
+				(hide yes)
+			)
+		)
+		(property "Description" ""
+			(at 74.93 105.41 0)
+			(effects
+				(font
+					(size 1.27 1.27)
+				)
+				(hide yes)
+			)
+		)
+		(pin "1"
+		)
+		(pin "1"
+		)
+		(instances
+			(project "Kicad_dev"
+				(path "/8104dfe2-da9a-40cd-b518-c622bfb26061"
+					(reference "U9")
+					(unit 1)
+				)

Commit message: Add repo of lib Kicad before analyzing...
Parts:
- removed U9: ~, CREPP_Battery_Holders:BK-18650-PC2_18650_Holder_THT [CREPP], symbol CREPP_Batteries:BK-18650-PC2_18650_Holder_THT [CREPP]
- added U25: LM358, Package_SO:SOIC-8_3.9x4.9mm_P1.27mm, symbol CREPP_AOP_SMT:LM358
Changed lines of the file:
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@@
 	)
 	(symbol
-		(lib_id "CREPP_Batteries:Battery_Cell")
-		(at 149.86 58.42 0)
-		(unit 1)
-		(exclude_from_sim no)
-		(in_bom yes)
-		(on_board yes)
-		(dnp no)
-		(fields_autoplaced yes)
-		(property "Reference" "BT1"
-			(at 153.67 55.3084 0)
-			(effects
-				(font
-					(size 1.27 1.27)
-				)
-				(justify left)
-			)
-		)
-		(property "Value" "Battery_Cell"
-			(at 153.67 57.8484 0)
-			(effects
-				(font
-					(size 1.27 1.27)
-				)
-				(justify left)
-			)
-		)
-		(property "Footprint" "BC501SM:MPD_BC501SM-TR"
-			(at 149.86 56.896 90)
-			(effects
-				(font
-					(size 1.27 1.27)
-				)
-				(hide yes)
-			)
-		)
-		(property "Datasheet" "~"
-			(at 149.86 56.896 90)
-			(effects
-				(font
-					(size 1.27 1.27)
-				)
-				(hide yes)
-			)
-		)
-		(property "Description" "Single-cell battery"
-			(at 149.86 58.42 0)
-			(effects
-				(font
-					(size 1.27 1.27)
-				)
-				(hide yes)
-			)
-		)
-		(pin "2"
-		)
-		(pin "1"
-		)
-		(instances
-			(project "Kicad_dev"
-				(path "/8104dfe2-da9a-40cd-b518-c622bfb26061"
-					(reference "BT1")
-					(unit 1)
-				)
-			)
-		)
-	)
-	(symbol
 		(lib_id "CREPP_Optocoupler:PC817_SMD")
 		(at 27.94 170.18 0)
@@
 	)
 	(symbol
+		(lib_id "CREPP_Batteries:Battery_Cell")
+		(at 153.67 69.85 0)
+		(unit 1)
+		(exclude_from_sim no)
+		(in_bom yes)
+		(on_board yes)
+		(dnp no)
+		(fields_autoplaced yes)
+		(property "Reference" "BT1"
+			(at 157.48 66.7384 0)
+			(effects
+				(font
+					(size 1.27 1.27)
+				)
+				(justify left)
+			)
+		)
+		(property "Value" "Battery_Cell"
+			(at 157.48 69.2784 0)
+			(effects
+				(font
+					(size 1.27 1.27)
+				)
+				(justify left)
+			)
+		)
+		(property "Footprint" "BC501SM:MPD_BC501SM-TR"
+			(at 153.67 68.326 90)
+			(effects
+				(font
+					(size 1.27 1.27)
+				)
+				(hide yes)
+			)
+		)
+		(property "Datasheet" "~"
+			(at 153.67 68.326 90)
+			(effects
+				(font
+					(size 1.27 1.27)
+				)
+				(hide yes)
+			)
+		)
+		(property "Description" "Single-cell battery"
+			(at 153.67 69.85 0)
+			(effects
+				(font
+					(size 1.27 1.27)
+				)
+				(hide yes)
+			)
+		)
+		(pin "1"
+		)
+		(pin "2"
+		)
+		(instances
+			(project "Kicad_dev"
+				(path "/8104dfe2-da9a-40cd-b518-c622bfb26061"
+					(reference "BT1")
+					(unit 1)
+				)
+			)
+		)
+	)
+	(symbol
 		(lib_id "CREPP_Buttons_THT:SW_DPST_x2")
 		(at -17.78 226.06 0)
@@
 	)
 	(symbol
+		(lib_id "CREPP_AOP_SMT:LM358")
+		(at 138.43 54.61 0)
+		(unit 1)
+		(exclude_from_sim no)
+		(in_bom yes)
+		(on_board yes)
+		(dnp no)
+		(fields_autoplaced yes)
+		(property "Reference" "U25"
+			(at 138.43 44.45 0)
+			(effects
+				(font
+					(size 1.27 1.27)
+				)
+			)
+		)
+		(property "Value" "LM358"
+			(at 138.43 46.99 0)
+			(effects
+				(font
+					(size 1.27 1.27)
+				)
+			)
+		)
+		(property "Footprint" "Package_SO:SOIC-8_3.9x4.9mm_P1.27mm"
+			(at 138.43 54.61 0)
+			(effects
+				(font
+					(size 1.27 1.27)
+				)
+				(hide yes)
+			)
+		)
+		(property "Datasheet" "http://www.ti.com/lit/ds/symlink/lm2904-n.pdf"
+			(at 138.43 54.61 0)
+			(effects
+				(font
+					(size 1.27 1.27)
+				)
+				(hide yes)
+			)
+		)
+		(property "Description" "Low-Power, Dual Operational Amplifiers, DIP-8/SOIC-8/TO-99-8"
+			(at 138.43 54.61 0)
+			(effects
+				(font
+					(size 1.27 1.27)
+				)
+				(hide yes)
+			)
+		)
+		(pin "8"
+		)
+		(pin "5"
+		)
+		(pin "7"
+		)
+		(pin "3"
+		)
+		(pin "2"
+		)
+		(pin "4"
+		)
+		(pin "1"
+		)
+		(pin "6"
+		)
+		(instances
+			(project "Kicad_dev"
+				(path "/8104dfe2-da9a-40cd-b518-c622bfb26061"
+					(reference "U25")
+					(unit 1)
+				)
+			)
+		)
+	)
+	(symbol
 		(lib_id "CREPP_MCU_STM32:STM32F723ZETx")
 		(at -22.86 369.57 0)
@@
 	)
 	(symbol
-		(lib_id "CREPP_Batteries:BK-18650-PC2_18650_Holder_THT [CREPP]")
-		(at 74.93 105.41 0)
-		(unit 1)
-		(exclude_from_sim no)
-		(in_bom yes)
-		(on_board yes)
-		(dnp no)
-		(fields_autoplaced yes)
-		(property "Reference" "U9"
-			(at 77.47 107.9499 0)
-			(effects
-				(font
-					(size 1.27 1.27)
-				)
-				(justify left)
-			)
-		)
-		(property "Value" "~"
-			(at 77.47 109.855 0)
-			(effects
-				(font
-					(size 1.27 1.27)
-				)
-				(justify left)
-			)
-		)
-		(property "Footprint" "CREPP_Battery_Holders:BK-18650-PC2_18650_Holder_THT [CREPP]"
-			(at 74.93 105.41 0)
-			(effects
-				(font
-					(size 1.27 1.27)
-				)
-				(hide yes)
-			)
-		)
-		(property "Datasheet" ""
-			(at 74.93 105.41 0)
-			(effects
-				(font
-					(size 1.27 1.27)
-				)
-				(hide yes)
-			)
-		)
-		(property "Description" ""
-			(at 74.93 105.41 0)
-			(effects
-				(font
-					(size 1.27 1.27)
-				)
-				(hide yes)
-			)
-		)
-		(pin "1"
-		)
-		(pin "1"
-		)
-		(instances
-			(project "Kicad_dev"
-				(path "/8104dfe2-da9a-40cd-b518-c622bfb26061"
-					(reference "U9")
-					(unit 1)
-				)
-			)
-		)
-	)
-	(symbol
 		(lib_id "CREPP_Logic:74HC04_THT")
 		(at 227.33 124.46 0)
@@
 	)
 	(symbol
+		(lib_id "CREPP_AOP_SMT:LM358")
+		(at 109.22 54.61 0)
+		(unit 3)
+		(exclude_from_sim no)
+		(in_bom yes)
+		(on_board yes)
+		(dnp no)
+		(fields_autoplaced yes)
+		(property "Reference" "U25"
+			(at 107.95 53.3399 0)
+			(effects
+				(font
+					(size 1.27 1.27)
+				)
+				(justify left)
+			)
+		)
+		(property "Value" "LM358"
+			(at 107.95 55.8799 0)
+			(effects
+				(font
+					(size 1.27 1.27)
+				)
+				(justify left)
+			)
+		)
+		(property "Footprint" "Package_SO:SOIC-8_3.9x4.9mm_P1.27mm"
+			(at 109.22 54.61 0)
+			(effects
+				(font
+					(size 1.27 1.27)
+				)
+				(hide yes)
+			)
+		)
+		(property "Datasheet" "http://www.ti.com/lit/ds/symlink/lm2904-n.pdf"
+			(at 109.22 54.61 0)
+			(effects
+				(font
+					(size 1.27 1.27)
+				)
+				(hide yes)
+			)
+		)
+		(property "Description" "Low-Power, Dual Operational Amplifiers, DIP-8/SOIC-8/TO-99-8"
+			(at 109.22 54.61 0)
+			(effects
+				(font
+					(size 1.27 1.27)
+				)
+				(hide yes)
+			)
+		)
+		(pin "8"
+		)
+		(pin "5"
+		)
+		(pin "7"
+		)
+		(pin "3"
+		)
+		(pin "2"
+		)
+		(pin "4"
+		)
+		(pin "1"
+		)
+		(pin "6"
+		)
+		(instances
+			(project "Kicad_dev"
+				(path "/8104dfe2-da9a-40cd-b518-c622bfb26061"
+					(reference "U25")
+					(unit 3)
+				)
+			)
+		)
+	)
+	(symbol
 		(lib_id "CREPP_Resistors:Resistor_THT_250mW (standard)")
 		(at 48.26 50.8 0)
@@
 				)
 			)
+		)
+	)
+	(symbol
+		(lib_id "CREPP_AOP_SMT:LM358")
+		(at 120.65 55.88 0)
+		(unit 2)
+		(exclude_from_sim no)
+		(in_bom yes)
+		(on_board yes)
+		(dnp no)
+		(fields_autoplaced yes)
+		(property "Reference" "U25"
+			(at 120.65 45.72 0)
+			(effects
+				(font
+					(size 1.27 1.27)
+				)
+			)
+		)
+		(property "Value" "LM358"
+			(at 120.65 48.26 0)
+			(effects
+				(font
+					(size 1.27 1.27)
+				)
+			)
+		)
+		(property "Footprint" "Package_SO:SOIC-8_3.9x4.9mm_P1.27mm"
+			(at 120.65 55.88 0)
+			(effects
+				(font
+					(size 1.27 1.27)
+				)
+				(hide yes)
+			)
+		)
+		(property "Datasheet" "http://www.ti.com/lit/ds/symlink/lm2904-n.pdf"
+			(at 120.65 55.88 0)
+			(effects
+				(font
+					(size 1.27 1.27)
+				)
+				(hide yes)
+			)
+		)
+		(property "Description" "Low-Power, Dual Operational Amplifiers, DIP-8/SOIC-8/TO-99-8"
+			(at 120.65 55.88 0)
+			(effects
+				(font
+					(size 1.27 1.27)
+				)
+				(hide yes)
+			)
+		)
+		(pin "8"
+		)
+		(pin "5"
+		)
+		(pin "7"
+		)
+		(pin "3"
+		)
+		(pin "2"
+		)
+		(pin "4"
+		)
+		(pin "1"
+		)
+		(pin "6"
+		)
+		(instances
+			(project "Kicad_dev"
+				(path "/8104dfe2-da9a-40cd-b518-c622bfb26061"
+					(reference "U25")
+					(unit 2)
+				)
+			)

Commit message: Add repo of lib Kicad before analyzing...
Parts:
- added BT2: Battery_Cell, CREPP_Battery_Holders:MPD_BC501SM-TR, symbol CREPP_Batteries:Battery_Cell
- added U9: ~, CREPP_Battery_Holders:BK-18650, symbol CREPP_Batteries:BK-18650-PC2_18650_Holder_THT
Changed lines of the file:
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@@
+	)
+	(symbol
+		(lib_name "Battery_Cell_1")
+		(lib_id "CREPP_Batteries:Battery_Cell")
+		(at 74.93 96.52 0)
+		(unit 1)
+		(exclude_from_sim no)
+		(in_bom yes)
+		(on_board yes)
+		(dnp no)
+		(fields_autoplaced yes)
+		(property "Reference" "BT2"
+			(at 78.74 93.4084 0)
+			(effects
+				(font
+					(size 1.27 1.27)
+				)
+				(justify left)
+			)
+		)
+		(property "Value" "Battery_Cell"
+			(at 78.74 95.9484 0)
+			(effects
+				(font
+					(size 1.27 1.27)
+				)
+				(justify left)
+			)
+		)
+		(property "Footprint" "CREPP_Battery_Holders:MPD_BC501SM-TR"
+			(at 74.93 94.996 90)
+			(effects
+				(font
+					(size 1.27 1.27)
+				)
+				(hide yes)
+			)
+		)
+		(property "Datasheet" "~"
+			(at 74.93 94.996 90)
+			(effects
+				(font
+					(size 1.27 1.27)
+				)
+				(hide yes)
+			)
+		)
+		(property "Description" "Single-cell battery"
+			(at 74.93 96.52 0)
+			(effects
+				(font
+					(size 1.27 1.27)
+				)
+				(hide yes)
+			)
+		)
+		(pin "2"
+		)
+		(pin "1"
+		)
+		(instances
+			(project "Kicad_dev"
+				(path "/8104dfe2-da9a-40cd-b518-c622bfb26061"
+					(reference "BT2")
+					(unit 1)
+				)
+			)
+		)
 	)
 	(symbol
@@
 					(unit 1)
 				)
+			)
+		)
+	)
+	(symbol
+		(lib_id "CREPP_Batteries:BK-18650-PC2_18650_Holder_THT")
+		(at 66.04 106.68 0)
+		(unit 1)
+		(exclude_from_sim no)
+		(in_bom yes)
+		(on_board yes)
+		(dnp no)
+		(fields_autoplaced yes)
+		(property "Reference" "U9"
+			(at 68.58 109.2199 0)
+			(effects
+				(font
+					(size 1.27 1.27)
+				)
+				(justify left)
+			)
+		)
+		(property "Value" "~"
+			(at 68.58 111.125 0)
+			(effects
+				(font
+					(size 1.27 1.27)
+				)
+				(justify left)
+			)
+		)
+		(property "Footprint" "CREPP_Battery_Holders:BK-18650"
+			(at 66.04 106.68 0)
+			(effects
+				(font
+					(size 1.27 1.27)
+				)
+				(hide yes)
+			)
+		)
+		(property "Datasheet" ""
+			(at 66.04 106.68 0)
+			(effects
+				(font
+					(size 1.27 1.27)
+				)
+				(hide yes)
+			)
+		)
+		(property "Description" ""
+			(at 66.04 106.68 0)
+			(effects
+				(font
+					(size 1.27 1.27)
+				)
+				(hide yes)
+			)
+		)
+		(pin "1"
+		)
+		(pin "1"
+		)
+		(instances
+			(project "Kicad_dev"
+				(path "/8104dfe2-da9a-40cd-b518-c622bfb26061"
+					(reference "U9")
+					(unit 1)
+				)

Commit message: Add repo of lib Kicad before analyzing...
Parts:
- removed JP1: Jumper_2.54mm_black, CREPP_Jumpers:Jumper_2.54mm_black, symbol CREPP_Jumpers:Jumper_2.54mm_black
- removed JP2: Jumper_2.54mm_red, CREPP_Jumpers:Jumper_2.54mm_red, symbol CREPP_Jumpers:Jumper_2.54mm_red
- removed JP3: Jumper_2.54mm_blue, CREPP_Jumpers:Jumper_2.54mm_blue, symbol CREPP_Jumpers:Jumper_2.54mm_blue
- added D5: 1N4148, Diode_THT:D_DO-35_SOD27_P7.62mm_Horizontal, symbol CREPP_Diodes_THT:1N4148
- added J7: Screw_Terminal_01x02_2.54mm, TerminalBlock_Phoenix:TerminalBlock_Phoenix_MPT-0,5-2-2.54_1x02_P2.54mm_Horizontal, symbol CREPP_Screw_Terminal:Screw_Terminal_01x02_2.54mm
- added JP1: Jumper_2.54mm_blue, CREPP_Jumpers:Jumper_2.54mm_blue, symbol CREPP_Jumpers:Jumper_2.54mm_blue
- added JP2: Jumper_2.54mm_green, CREPP_Jumpers:Jumper_2.54mm_green, symbol CREPP_Jumpers:Jumper_2.54mm_green
- added U26: TP4056, CREPP_BMS:SOP127P600X175-9N, symbol CREPP_BMS:TP4056
