File: Kicad_dev/Kicad_dev.kicad_sch (KiCad schematic)
At the start: 62 parts, among them J1 Conn_01x02_Pin, J2 Conn_01x02_Pin, J3 Conn_01x02_Pin, J4 530470510_Picoblade, J5 Connecteur_SMA, J6 BNC, J7 Screw_Terminal_01x02_2.54mm, Q1 IRF540N, SW1 RotaryEncoder_Switch, SW2 RotaryEncoder_Switch, SW3 SW_DPST_x2, SW4 SW_DPST_x2, U1 COM-09032, U11 MAX-8Q, U12 LM317_TO-220, U13 LM7805_TO220, U14 DHT11, U15 DHT11, U17 ATmega328-A, U18 ATmega328-P, U19 STM32F030CCTx, U2 LM317_SOT-223, U20 STM32F446VETx, U21 STM32F723ZETx, U22 MPU-6050, U23 DS1307+, U24 DS3231M, U25 LM358, U26 TP4056, U3 74HC04, U4 L293D, U5 LM358, U6 PC817_SMD, U7 PC817_THT, U8 NEO-M8Q

Commit message: Add repo of lib Kicad before analyzing...
Parts:
- removed U16: ~, symbol CREPP_Temperature_sensors:BME280_Breakout
- added J10: Screw_Terminal_01x05_2.54mm, TerminalBlock_Phoenix:TerminalBlock_Phoenix_MPT-0,5-5-2.54_1x05_P2.54mm_Horizontal, symbol CREPP_Screw_Terminal:Screw_Terminal_01x05_2.54mm
- added J8: Screw_Terminal_01x03_2.54mm, TerminalBlock_Phoenix:TerminalBlock_Phoenix_MPT-0,5-3-2.54_1x03_P2.54mm_Horizontal, symbol CREPP_Screw_Terminal:Screw_Terminal_01x03_2.54mm
- added J9: Screw_Terminal_01x04_2.54mm, TerminalBlock_Phoenix:TerminalBlock_Phoenix_MPT-0,5-4-2.54_1x04_P2.54mm_Horizontal, symbol CREPP_Screw_Terminal:Screw_Terminal_01x04_2.54mm
- added U27: ~, CREPP_Temperature_sensors:BME280_Breakout, symbol CREPP_Temperature_sensors:BME280_Breakout
Changed lines of the file:
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@@
+	)
+	(symbol
+		(lib_id "CREPP_Screw_Terminal:Screw_Terminal_01x03_2.54mm")
+		(at -60.96 36.83 0)
+		(unit 1)
+		(exclude_from_sim no)
+		(in_bom yes)
+		(on_board yes)
+		(dnp no)
+		(fields_autoplaced yes)
+		(property "Reference" "J8"
+			(at -57.15 35.5599 0)
+			(effects
+				(font
+					(size 1.27 1.27)
+				)
+				(justify left)
+			)
+		)
+		(property "Value" "Screw_Terminal_01x03_2.54mm"
+			(at -57.15 38.0999 0)
+			(effects
+				(font
+					(size 1.27 1.27)
+				)
+				(justify left)
+			)
+		)
+		(property "Footprint" "TerminalBlock_Phoenix:TerminalBlock_Phoenix_MPT-0,5-3-2.54_1x03_P2.54mm_Horizontal"
+			(at -60.96 36.83 0)
+			(effects
+				(font
+					(size 1.27 1.27)
+				)
+				(hide yes)
+			)
+		)
+		(property "Datasheet" "~"
+			(at -60.96 36.83 0)
+			(effects
+				(font
+					(size 1.27 1.27)
+				)
+				(hide yes)
+			)
+		)
+		(property "Description" "Generic screw terminal, single row, 01x03, script generated (kicad-library-utils/schlib/autogen/connector/)"
+			(at -60.96 36.83 0)
+			(effects
+				(font
+					(size 1.27 1.27)
+				)
+				(hide yes)
+			)
+		)
+		(pin "3"
+		)
+		(pin "2"
+		)
+		(pin "1"
+		)
+		(instances
+			(project "Kicad_dev"
+				(path "/8104dfe2-da9a-40cd-b518-c622bfb26061"
+					(reference "J8")
+					(unit 1)
+				)
+			)
+		)
+	)
+	(symbol
+		(lib_id "CREPP_Screw_Terminal:Screw_Terminal_01x04_2.54mm")
+		(at -60.96 46.99 0)
+		(unit 1)
+		(exclude_from_sim no)
+		(in_bom yes)
+		(on_board yes)
+		(dnp no)
+		(fields_autoplaced yes)
+		(property "Reference" "J9"
+			(at -57.15 46.9899 0)
+			(effects
+				(font
+					(size 1.27 1.27)
+				)
+				(justify left)
+			)
+		)
+		(property "Value" "Screw_Terminal_01x04_2.54mm"
+			(at -57.15 49.5299 0)
+			(effects
+				(font
+					(size 1.27 1.27)
+				)
+				(justify left)
+			)
+		)
+		(property "Footprint" "TerminalBlock_Phoenix:TerminalBlock_Phoenix_MPT-0,5-4-2.54_1x04_P2.54mm_Horizontal"
+			(at -60.96 46.99 0)
+			(effects
+				(font
+					(size 1.27 1.27)
+				)
+				(hide yes)
+			)
+		)
+		(property "Datasheet" "~"
+			(at -60.96 46.99 0)
+			(effects
+				(font
+					(size 1.27 1.27)
+				)
+				(hide yes)
+			)
+		)
+		(property "Description" "Generic screw terminal, single row, 01x04, script generated (kicad-library-utils/schlib/autogen/connector/)"
+			(at -60.96 46.99 0)
+			(effects
+				(font
+					(size 1.27 1.27)
+				)
+				(hide yes)
+			)
+		)
+		(pin "4"
+		)
+		(pin "1"
+		)
+		(pin "3"
+		)
+		(pin "2"
+		)
+		(instances
+			(project "Kicad_dev"
+				(path "/8104dfe2-da9a-40cd-b518-c622bfb26061"
+					(reference "J9")
+					(unit 1)
+				)
+			)
+		)
 	)
 	(symbol
@@
 	)
 	(symbol
-		(lib_id "CREPP_Temperature_sensors:BME280_Breakout")
-		(at 163.83 185.42 0)
-		(unit 1)
-		(exclude_from_sim no)
-		(in_bom yes)
-		(on_board yes)
-		(dnp no)
-		(fields_autoplaced yes)
-		(property "Reference" "U16"
-			(at 175.26 186.6899 0)
-			(effects
-				(font
-					(size 1.27 1.27)
-				)
-				(justify left)
-			)
-		)
-		(property "Value" "~"
-			(at 175.26 188.595 0)
-			(effects
-				(font
-					(size 1.27 1.27)
-				)
-				(justify left)
-			)
-		)
-		(property "Footprint" ""
-			(at 163.83 185.42 0)
-			(effects
-				(font
-					(size 1.27 1.27)
-				)
-				(hide yes)
-			)
-		)
-		(property "Datasheet" ""
-			(at 163.83 185.42 0)
-			(effects
-				(font
-					(size 1.27 1.27)
-				)
-				(hide yes)
-			)
-		)
-		(property "Description" ""
-			(at 163.83 185.42 0)
-			(effects
-				(font
-					(size 1.27 1.27)
-				)
-				(hide yes)
-			)
-		)
-		(instances
-			(project "Kicad_dev"
-				(path "/8104dfe2-da9a-40cd-b518-c622bfb26061"
-					(reference "U16")
-					(unit 1)
-				)
-			)
-		)
-	)
-	(symbol
 		(lib_id "CREPP_DIP:DIP-8-Device")
 		(at 50.8 97.79 0)
@@
 				(path "/8104dfe2-da9a-40cd-b518-c622bfb26061"
 					(reference "V1")
+					(unit 1)
+				)
+			)
+		)
+	)
+	(symbol
+		(lib_name "BME280_Breakout_1")
+		(lib_id "CREPP_Temperature_sensors:BME280_Breakout")
+		(at 161.29 201.93 0)
+		(unit 1)
+		(exclude_from_sim no)
+		(in_bom yes)
+		(on_board yes)
+		(dnp no)
+		(fields_autoplaced yes)
+		(property "Reference" "U27"
+			(at 172.72 203.1999 0)
+			(effects
+				(font
+					(size 1.27 1.27)
+				)
+				(justify left)
+			)
+		)
+		(property "Value" "~"
+			(at 172.72 205.105 0)
+			(effects
+				(font
+					(size 1.27 1.27)
+				)
+				(justify left)
+			)
+		)
+		(property "Footprint" "CREPP_Temperature_sensors:BME280_Breakout"
+			(at 161.29 201.93 0)
+			(effects
+				(font
+					(size 1.27 1.27)
+				)
+				(hide yes)
+			)
+		)
+		(property "Datasheet" ""
+			(at 161.29 201.93 0)
+			(effects
+				(font
+					(size 1.27 1.27)
+				)
+				(hide yes)
+			)
+		)
+		(property "Description" ""
+			(at 161.29 201.93 0)
+			(effects
+				(font
+					(size 1.27 1.27)
+				)
+				(hide yes)
+			)
+		)
+		(instances
+			(project "Kicad_dev"
+				(path "/8104dfe2-da9a-40cd-b518-c622bfb26061"
+					(reference "U27")
 					(unit 1)
 				)
@@
 					(unit 1)
 				)
+			)
+		)
+	)
+	(symbol
+		(lib_id "CREPP_Screw_Terminal:Screw_Terminal_01x05_2.54mm")
+		(at -113.03 46.99 0)
+		(unit 1)
+		(exclude_from_sim no)
+		(in_bom yes)
+		(on_board yes)
+		(dnp no)
+		(fields_autoplaced yes)
+		(property "Reference" "J10"
+			(at -109.22 45.7199 0)
+			(effects
+				(font
+					(size 1.27 1.27)
+				)
+				(justify left)
+			)
+		)
+		(property "Value" "Screw_Terminal_01x05_2.54mm"
+			(at -109.22 48.2599 0)
+			(effects
+				(font
+					(size 1.27 1.27)
+				)
+				(justify left)
+			)
+		)
+		(property "Footprint" "TerminalBlock_Phoenix:TerminalBlock_Phoenix_MPT-0,5-5-2.54_1x05_P2.54mm_Horizontal"
+			(at -113.03 46.99 0)
+			(effects
+				(font
+					(size 1.27 1.27)
+				)
+				(hide yes)
+			)
+		)
+		(property "Datasheet" "~"
+			(at -113.03 46.99 0)
+			(effects
+				(font
+					(size 1.27 1.27)
+				)
+				(hide yes)
+			)
+		)
+		(property "Description" "Generic screw terminal, single row, 01x05, script generated (kicad-library-utils/schlib/autogen/connector/)"
+			(at -113.03 46.99 0)
+			(effects
+				(font
+					(size 1.27 1.27)
+				)
+				(hide yes)
+			)
+		)
+		(pin "1"
+		)
+		(pin "5"
+		)
+		(pin "4"
+		)
+		(pin "3"
+		)
+		(pin "2"
+		)
+		(instances
+			(project "Kicad_dev"
+				(path "/8104dfe2-da9a-40cd-b518-c622bfb26061"
+					(reference "J10")
+					(unit 1)
+				)

Commit message: Add repo of lib Kicad before analyzing...
Parts:
- removed BT1: Battery_Cell, BC501SM:MPD_BC501SM-TR, symbol CREPP_Batteries:Battery_Cell
- removed BT2: Battery_Cell, CREPP_Battery_Holders:MPD_BC501SM-TR, symbol CREPP_Batteries:Battery_Cell
- removed U9: ~, CREPP_Battery_Holders:BK-18650, symbol CREPP_Batteries:BK-18650-PC2_18650_Holder_THT
- added BT2: Battery_Cell, CREPP_Batteries_holders:MPD_BC501SM-TR, symbol CREPP_Batteries_holders:Battery_Cell
- added Q2: 2N7000_THT, Package_TO_SOT_THT:TO-92_Inline, symbol CREPP_Transistors_NMOS_THT:2N7000_THT
- added Q3: 2N7002, Package_TO_SOT_SMD:SOT-23, symbol CREPP_Transistors_NMOS_CMS:2N7002
- added U9: ~, CREPP_Batteries_holders:BK-18650, symbol CREPP_Batteries_holders:BK-18650-PC2_18650_Holder_THT
Other:
- moved on the sheet: SW3A, SW3B, SW4A, SW4B, U19, U20, U21, U6, U7
