File: Kicad_dev/Kicad_dev.kicad_pcb (KiCad board)
At the start: 2 copper layers, 29 parts, among them J1 Conn_01x02_Pin, J2 Conn_01x02_Pin, J3 Conn_01x02_Pin, J5 Conn_Coaxial, J6 BNC, J7 BNC, J8 BNC, J9 BNC, Q1 IRF540N, SW1 RotaryEncoder_Switch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

Commit message: Add
Parts:
- removed U2: COM-09032, CREPP_Joysticks:XDCR_COM-09032
- added J4: 530470510_Picoblade, CREPP_Connector_Picoblade:MOLEX_530470510, F.Cu at (168.9, 57.8)
- moved U4 97.2 mm to (154.4, 113.7)
- moved S1 74.8 mm to (167.6, 115.1)
- moved S2 74.8 mm to (167.6, 122.3)
- moved S3 74.8 mm to (167.6, 129.5)
- moved U8 70.1 mm to (144.6, 120.3)
- moved J1 62.5 mm to (157.8, 102.9)
- moved J2 62.5 mm to (162.5, 102.9)
- moved J3 62.5 mm to (167.1, 102.9)
- moved HS1 43.2 mm to (137.7, 136.5)
- moved U1 39.4 mm to (95.0, 112.5)
- moved U3 38.4 mm to (157.6, 83.2)
- moved JP1 35.5 mm to (162.4, 76.2)
- moved JP2 35.5 mm to (166.1, 76.2)
- moved JP3 35.5 mm to (169.7, 76.2)
- moved Q1 35.5 mm to (163.8, 72.3)
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
Commit message: Add
Parts:
- added U12: COM-09032, CREPP_Joysticks:XDCR_COM-09032, F.Cu at (69.6, 96.5)
- added U2: COM-09032, CREPP_Joysticks:XDCR_COM-09032, F.Cu at (41.5, 96.5)

Commit message: Add
Parts:
- removed J7, J8, J9: BNC, Connector_Coaxial:BNC_Amphenol_B6252HB-NPP3G-50_Horizontal
- J5: value Conn_Coaxial -> Connecteur_SMA
- moved J6 16.0 mm to (101.6, 67.8)

Commit message: Add
Parts:
- added OLED1: ~, CREPP_Screens:SSD1306_OLED_Display(128x64), F.Cu at (61.9, 38.7)
- added R1: 10k, Resistor_THT:R_Axial_DIN0309_L9.0mm_D3.2mm_P12.70mm_Horizontal, F.Cu at (49.2, 67.4)
- added R2: 10k, Resistor_THT:R_Axial_DIN0207_L6.3mm_D2.5mm_P7.62mm_Horizontal, F.Cu at (65.0, 67.1)
- J6: footprint Connector_Coaxial:BNC_Amphenol_B6252HB-NPP3G-50_Horizontal -> CREPP_BNC:BNC_Amphenol_B6252HB-NPP3G-50_Horizontal
- moved J6 9.56 mm to (99.8, 58.4)
- moved U2 0.91 mm to (40.9, 95.8)

Commit message: Add repo of lib Kicad before analyzing...
Parts:
- removed U1: ~, CREPP_Screens:SSD1306_OLED_Display(128x64)
- moved R1 111.3 mm to (151.2, 111.9)
- moved J4 104.8 mm to (90.5, 127.4)
- moved OLED1 92.0 mm to (152.7, 53.5)
- moved R2 81.6 mm to (119.1, 128.3)
- moved V1 71.3 mm to (155.7, 116.4)
- moved U7 67.5 mm to (119.1, 115.7)
- moved Q1 67.5 mm to (120.7, 124.2)
- moved U3 63.9 mm to (101.0, 112.9)
- moved U2 62.7 mm to (96.3, 66.3)
- moved U12 62.6 mm to (124.4, 66.3)
- moved J6 56.9 mm to (90.6, 114.6)
- moved U6 55.9 mm to (88.8, 121.2)
- moved JP1 51.9 mm to (156.8, 127.8)
- moved JP2 51.9 mm to (160.4, 127.8)
- moved JP3 51.9 mm to (164.1, 127.8)
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
Commit message: Add repo of lib Kicad before analyzing...
Parts:
- removed OLED1: ~, CREPP_Screens:SSD1306_OLED_Display(128x64)
- added U1: COM-09032, CREPP_Joysticks:XDCR_COM-09032_V2, F.Cu at (159.0, 61.7)

Commit message: Add repo of lib Kicad before analyzing...
Parts:
- added OLED1: ~, CREPP_Screens:SSD1306_OLED_Display_VIRTUAL_128_64, F.Cu at (197.6, 93.5)
Changed lines of the file:
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@@
+		)
+	)
+	(footprint "CREPP_Screens:SSD1306_OLED_Display_VIRTUAL_128_64"
+		(layer "F.Cu")
+		(at 197.612 93.472)
+		(descr "Display 0.96\" OLED 128x64 pixel with SSD1306 controller and I2C interface")
+		(tags "display OLED SSD1306 128x64")
+		(property "Reference" "OLED1"
+			(at -0.2286 10.8712 0)
+			(layer "F.SilkS")
+			(hide yes)
+			(effects
+				(font
+					(size 1 1)
+					(thickness 0.15)
+				)
+			)
+		)
+		(property "Value" "~"
+			(at -7.874 4.699 0)
+			(layer "F.Fab")
+			(effects
+				(font
+					(size 1 1)
+					(thickness 0.15)
+				)
+			)
+		)
+		(property "Footprint" "CREPP_Screens:SSD1306_OLED_Display_VIRTUAL_128_64"
+			(at 0 0 0)
+			(unlocked yes)
+			(layer "F.Fab")
+			(hide yes)
+			(effects
+				(font
+					(size 1.27 1.27)
+				)
+			)
+		)
+		(property "Datasheet" ""
+			(at 0 0 0)
+			(unlocked yes)
+			(layer "F.Fab")
+			(hide yes)
+			(effects
+				(font
+					(size 1.27 1.27)
+				)
+			)
+		)
+		(property "Description" ""
+			(at 0 0 0)
+			(unlocked yes)
+			(layer "F.Fab")
+			(hide yes)
+			(effects
+				(font
+					(size 1.27 1.27)
+				)
+			)
+		)
+		(sheetname "Racine")
+		(sheetfile "Kicad_dev.kicad_sch")
+		(attr through_hole)
+		(fp_line
+			(start -13.716 -1.397)
+			(end 13.716 -1.397)
+			(stroke
+				(width 0.12)
+				(type solid)
+			)
+			(layer "Dwgs.User")
+		)
+		(fp_line
+			(start -13.716 3.81)
+			(end 13.716 3.81)
+			(stroke
+				(width 0.12)
+				(type solid)
+			)
+			(layer "Dwgs.User")
+		)
+		(fp_line
+			(start -13.716 20.701)
+			(end 13.716 20.701)
+			(stroke
+				(width 0.12)
+				(type solid)
+			)
+			(layer "Dwgs.User")
+		)
+		(fp_line
+			(start -13.716 25.781)
+			(end -13.589 -1.397)
+			(stroke
+				(width 0.12)
+				(type solid)
+			)
+			(layer "Dwgs.User")
+		)
+		(fp_line
+			(start 13.716 25.781)
+			(end -13.716 25.781)
+			(stroke
+				(width 0.12)
+				(type solid)
+			)
+			(layer "Dwgs.User")
+		)
+		(fp_line
+			(start 13.716 25.781)
+			(end 13.716 -1.397)
+			(stroke
+				(width 0.12)
+				(type solid)
+			)
+			(layer "Dwgs.User")
+		)
+		(fp_circle
+			(center -11.2268 23.7744)
+			(end -9.8044 23.7744)
+			(stroke
+				(width 0.1)
+				(type default)
+			)
+			(fill none)
+			(layer "Dwgs.User")
+		)
+		(fp_circle
+			(center -11.176 0.6096)
+			(end -9.7536 0.6096)
+			(stroke
+				(width 0.1)
+				(type default)
+			)
+			(fill none)
+			(layer "Dwgs.User")
+		)
+		(fp_circle
+			(center 11.176 0.6604)
+			(end 12.5984 0.6604)
+			(stroke
+				(width 0.1)
+				(type default)
+			)
+			(fill none)
+			(layer "Dwgs.User")
+		)
+		(fp_circle
+			(center 11.2268 23.7744)
+			(end 12.6492 23.7744)
+			(stroke
+				(width 0.1)
+				(type default)
+			)
+			(fill none)
+			(layer "Dwgs.User")
+		)
+		(fp_line
+			(start -5.08 -1.27)
+			(end 5.08 -1.27)
+			(stroke
+				(width 0.1)
+				(type solid)
+			)
+			(layer "F.Fab")
+		)
+		(fp_line
+			(start -5.08 0.635)
+			(end -5.08 -1.27)
+			(stroke
+				(width 0.1)
+				(type solid)
+			)
+			(layer "F.Fab")
+		)
+		(fp_line
+			(start -4.445 1.27)
+			(end -5.08 0.635)
+			(stroke
+				(width 0.1)
+				(type solid)
+			)
+			(layer "F.Fab")
+		)
+		(fp_line
+			(start 5.08 -1.27)
+			(end 5.08 1.27)
+			(stroke
+				(width 0.1)
+				(type solid)
+			)
+			(layer "F.Fab")
+		)
+		(fp_line
+			(start 5.08 1.27)
+			(end -4.445 1.27)
+			(stroke
+				(width 0.1)
+				(type solid)
+			)
+			(layer "F.Fab")
+		)
+		(model "${KICAD8_3RD_PARTY}/3dmodels/com_github_crepp_library/CREPP_Screens/SSD1306_OLED_Display(128x64).step"
+			(offset
+				(xyz 0 -12 0)
+			)
+			(scale
+				(xyz 1 1 1)
+			)
+			(rotate
+				(xyz 0 0 0)
+			)
 		)
 	)

Commit message: Add repo of lib Kicad before analyzing...
Parts:
- removed U12, U2: COM-09032, CREPP_Joysticks:XDCR_COM-09032
- U1: footprint CREPP_Joysticks:XDCR_COM-09032_V2 -> CREPP_Joysticks_SW:XDCR_COM-09032
- moved OLED1 153.9 mm to (45.4, 70.3)
- moved U1 105.3 mm to (53.9, 54.5)
