File: Kicad_dev/Kicad_dev.kicad_pcb (KiCad board)
At the start: 2 copper layers, 29 parts, among them J1 Conn_01x02_Pin, J2 Conn_01x02_Pin, J3 Conn_01x02_Pin, J4 530470510_Picoblade, J5 Connecteur_SMA, J6 BNC, Q1 IRF540N, SW1 RotaryEncoder_Switch, SW2 RotaryEncoder_Switch, U1 COM-09032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

Commit message: Add repo of lib Kicad before analyzing...
Parts:
- added D1: LED_5mm_THT, LED_SMD:LED_0603_1608Metric, F.Cu at (152.6, 68.8)
- added D2: LED_5mm_THT, LED_THT:LED_D5.0mm, F.Cu at (148.6, 63.8)
- added D3: LED_5mm_THT, LED_SMD:LED_0805_2012Metric, F.Cu at (148.4, 69.1)

Commit message: Add repo of lib Kicad before analyzing...
Parts:
- added C1: Supercapacitors_D10mm_H20mm, CREPP_Capacitors_THT:C_Radial_D10.0mm_H20.0mm_P5.00mm, F.Cu at (112.7, 120.6)
- added C2: Supercapacitors_D10mm_H20mm, CREPP_Capacitors_THT:C_Radial_D10.0mm_H20.0mm_P5.00mm, F.Cu at (112.9, 133.6)
- added R3: R_0805, Resistor_SMD:R_0805_2012Metric, F.Cu at (92.7, 110.8)
- added U12: LM317_TO-220, Package_TO_SOT_THT:TO-220-3_Vertical, F.Cu at (112.7, 106.8)
- added U13: LM7805_TO220, Package_TO_SOT_THT:TO-220-3_Vertical, F.Cu at (112.7, 112.8)
- added U2: LM317_SOT-223, Package_TO_SOT_SMD:SOT-223-3_TabPin2, F.Cu at (142.1, 80.5)
- moved OLED1 105.2 mm to (142.0, 112.2)
- moved D2 78.0 mm to (100.2, 124.9)
- moved D1 74.9 mm to (92.6, 113.6)
- moved U1 70.8 mm to (123.2, 69.3)
- moved D3 67.8 mm to (92.8, 107.8)
- moved S1 67.1 mm to (94.1, 88.3)
- moved S2 67.1 mm to (94.1, 95.5)
- moved S3 67.1 mm to (94.1, 102.7)
- moved JP1 61.3 mm to (99.5, 106.0)
- moved JP3 61.3 mm to (106.8, 106.0)
- moved JP2 61.3 mm to (103.2, 106.0)
- moved J4 58.1 mm to (144.7, 106.5)
- moved U6 58.1 mm to (142.9, 100.2)
- moved SERVO_SG1 45.2 mm to (80.1, 100.5)
- moved J1 33.2 mm to (123.3, 121.5)
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
Commit message: Add repo of lib Kicad before analyzing...
Parts:
- added D4: SS24, Diode_SMD:D_SMA, F.Cu at (160.5, 86.0)
- added RV1: R_Potentiometer, Potentiometer_THT:Potentiometer_Alps_RK163_Single_Horizontal, F.Cu at (176.0, 69.0)

Commit message: Add repo of lib Kicad before analyzing...
Parts:
- added R4: LDR03, OptoDevice:R_LDR_7x6mm_P5.1mm_Vertical, F.Cu at (54.6, 68.8)
- added U14: DHT11, Sensor:Aosong_DHT11_5.5x12.0_P2.54mm, F.Cu at (56.3, 54.5)
- added U15: DHT11, Sensor:Aosong_DHT11_5.5x12.0_P2.54mm, F.Cu at (63.6, 54.5)

Commit message: Add repo of lib Kicad before analyzing...
Parts:
- added SW3: SW_DPST_x2, Button_Switch_SMD:SW_SPST_PTS645, F.Cu at (58.5, 118.1)
- added SW4: SW_DPST_x2, Button_Switch_THT:SW_PUSH_6mm_H4.3mm, F.Cu at (60.8, 91.6)
- added U17: ATmega328-A, Package_QFP:TQFP-32_7x7mm_P0.8mm, F.Cu at (58.8, 108.4)
- added U18: ATmega328-P, Package_DIP:DIP-28_W7.62mm, F.Cu at (25.2, 80.3)
- added U19: STM32F030CCTx, Package_QFP:LQFP-48_7x7mm_P0.5mm, F.Cu at (64.5, 83.9)
- added U20: STM32F446VETx, Package_QFP:LQFP-100_14x14mm_P0.5mm, F.Cu at (43.7, 111.8)
- added U21: STM32F723ZETx, Package_QFP:LQFP-144_20x20mm_P0.5mm, F.Cu at (46.6, 90.4)
- added U22: MPU-6050, Sensor_Motion:InvenSense_QFN-24_4x4mm_P0.5mm, F.Cu at (26.8, 118.5)

Commit message: Add repo of lib Kicad before analyzing...
Parts:
- added BT1: Battery_Cell, BC501SM:MPD_BC501SM-TR, F.Cu at (172.0, 99.6)
- added U23: DS1307+, Package_DIP:DIP-8_W7.62mm_Socket, F.Cu at (176.8, 110.0)
- added U24: DS3231M, Package_SO:SOIC-16W_7.5x10.3mm_P1.27mm, F.Cu at (168.3, 113.9)

Commit message: Add repo of lib Kicad before analyzing...
Parts:
- added U25: ~, CREPP_Battery_Holders:BK-18650-PC2_18650_Holder_THT [CREPP], F.Cu at (107.4, 34.3)

Commit message: Add repo of lib Kicad before analyzing...
Parts:
- removed U25: ~, CREPP_Battery_Holders:BK-18650-PC2_18650_Holder_THT [CREPP]
- added U9: ~, CREPP_Battery_Holders:BK-18650-PC2_18650_Holder_THT [CREPP], F.Cu at (75.9, 26.4)
