File: Kicad_dev/Kicad_dev.kicad_pcb (KiCad board)
At the start: 2 copper layers, 55 parts, among them J1 Conn_01x02_Pin, J2 Conn_01x02_Pin, J3 Conn_01x02_Pin, J4 530470510_Picoblade, J5 Connecteur_SMA, J6 BNC, Q1 IRF540N, SW1 RotaryEncoder_Switch, SW2 RotaryEncoder_Switch, SW3 SW_DPST_x2, SW4 SW_DPST_x2, U1 COM-09032, U11 MAX-8Q, U12 LM317_TO-220, U13 LM7805_TO220, U14 DHT11, U15 DHT11, U17 ATmega328-A, U18 ATmega328-P, U19 STM32F030CCTx, U2 LM317_SOT-223, U20 STM32F446VETx, U21 STM32F723ZETx, U22 MPU-6050, U23 DS1307+, U24 DS3231M, U3 74HC04, U4 L293D, U5 LM358, U6 PC817_SMD, U7 PC817_THT, U8 NEO-M8Q

Commit message: Add repo of lib Kicad before analyzing...
Parts:
- added U25: LM358, Package_SO:SOIC-8_3.9x4.9mm_P1.27mm, F.Cu at (162.9, 54.2)

Commit message: Add repo of lib Kicad before analyzing...
Parts:
- added BT2: Battery_Cell, CREPP_Battery_Holders:MPD_BC501SM-TR, F.Cu at (34.0, 63.3)
- U9: footprint CREPP_Battery_Holders:BK-18650-PC2_18650_Holder_THT [CREPP] -> CREPP_Battery_Holders:BK-18650
- moved BT1 147.8 mm to (34.0, 46.7)
- moved JP1 36.2 mm to (86.9, 140.0)
- moved U9 9.94 mm to (66.0, 27.2)

Commit message: Add repo of lib Kicad before analyzing...
Parts:
- removed JP3: Jumper_2.54mm_blue, CREPP_Jumpers:Jumper_2.54mm_blue
- added D5: 1N4148, Diode_THT:D_DO-35_SOD27_P7.62mm_Horizontal, F.Cu at (113.9, 31.2)
- added J7: Screw_Terminal_01x02_2.54mm, TerminalBlock_Phoenix:TerminalBlock_Phoenix_MPT-0,5-2-2.54_1x02_P2.54mm_Horizontal, F.Cu at (124.2, 37.1)
- added U26: TP4056, CREPP_BMS:SOP127P600X175-9N, F.Cu at (117.4, 36.3)
- JP1: value Jumper_2.54mm_black -> Jumper_2.54mm_blue; footprint CREPP_Jumpers:Jumper_2.54mm_black -> CREPP_Jumpers:Jumper_2.54mm_blue
- JP2: value Jumper_2.54mm_red -> Jumper_2.54mm_green; footprint CREPP_Jumpers:Jumper_2.54mm_red -> CREPP_Jumpers:Jumper_2.54mm_green

Commit message: Add repo of lib Kicad before analyzing...
Parts:
- added J10: Screw_Terminal_01x05_2.54mm, TerminalBlock_Phoenix:TerminalBlock_Phoenix_MPT-0,5-5-2.54_1x05_P2.54mm_Horizontal, F.Cu at (180.4, 54.6)
- added J8: Screw_Terminal_01x03_2.54mm, TerminalBlock_Phoenix:TerminalBlock_Phoenix_MPT-0,5-3-2.54_1x03_P2.54mm_Horizontal, F.Cu at (197.9, 41.3)
- added J9: Screw_Terminal_01x04_2.54mm, TerminalBlock_Phoenix:TerminalBlock_Phoenix_MPT-0,5-4-2.54_1x04_P2.54mm_Horizontal, F.Cu at (195.6, 54.6)
- added U27: ~, CREPP_Temperature_sensors:BME280_Breakout, F.Cu at (187.1, 40.1)

Commit message: Add repo of lib Kicad before analyzing...
Parts:
- removed BT1: Battery_Cell, BC501SM:MPD_BC501SM-TR
- removed RV1: R_Potentiometer, Potentiometer_THT:Potentiometer_Alps_RK163_Single_Horizontal
- added Q2: 2N7000_THT, Package_TO_SOT_THT:TO-92_Inline, F.Cu at (104.9, 163.1)
- added Q3: 2N7002, Package_TO_SOT_SMD:SOT-23, F.Cu at (111.9, 162.2)
- BT2: footprint CREPP_Battery_Holders:MPD_BC501SM-TR -> CREPP_Batteries_holders:MPD_BC501SM-TR
- U9: footprint CREPP_Battery_Holders:BK-18650 -> CREPP_Batteries_holders:BK-18650
- moved BT2 127.6 mm to (146.3, 123.9)
- moved J7 124.1 mm to (168.7, 152.9)
- moved U17 122.2 mm to (168.7, 55.2)
- moved U26 114.7 mm to (117.5, 150.9)
- moved SW3 110.7 mm to (155.6, 65.0)
- moved J10 108.6 mm to (138.6, 154.8)
- moved U20 105.9 mm to (145.3, 141.5)
- moved J8 99.5 mm to (168.7, 136.3)
- moved R4 95.9 mm to (114.4, 143.8)
- moved U25 91.2 mm to (86.7, 104.3)
- moved D5 90.9 mm to (84.0, 117.0)
- moved U18 90.6 mm to (114.0, 98.3)
- moved U14 88.2 mm to (69.4, 141.7)
- moved U15 88.2 mm to (76.6, 141.7)
- moved D4 88.0 mm to (86.5, 133.6)
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
Commit message: Add repo of lib Kicad before analyzing...
Parts:
- added RV1: R_Potentiometer, Potentiometer_THT:Potentiometer_Alps_RK163_Single_Horizontal, F.Cu at (205.7, 115.7)
- added TP1: MM8130-2600, CREPP_Connectors_MURATA:MM8130-2600, F.Cu at (166.9, 119.6)
- moved J5 41.1 mm to (212.1, 144.3)

Commit message: Add repo of lib Kicad before analyzing...
Parts:
- added S4: ~, CREPP_Spacers:Spacer_M3_FF_20mm, F.Cu at (135.0, 153.7)
- S1: footprint CREPP_Spacers:Spacer_M3_MF_05mm -> CREPP_Spacers:Spacer_M3_FF_05mm
- S2: footprint CREPP_Spacers:Spacer_M3_MF_05mm -> CREPP_Spacers:Spacer_M3_FF_10mm
- S3: footprint CREPP_Spacers:Spacer_M3_MF_05mm -> CREPP_Spacers:Spacer_M3_FF_15mm
- moved J5 165.3 mm to (46.8, 140.9)
- moved OLED1 144.4 mm to (64.9, 130.4)
- moved J9 135.9 mm to (60.3, 151.2)
- moved U27 126.8 mm to (79.9, 121.1)
- moved U11 108.2 mm to (106.5, 151.2)
- moved J7 105.3 mm to (64.3, 138.9)
- moved Q2 104.7 mm to (141.8, 65.1)
- moved Q3 104.7 mm to (148.8, 64.3)
- moved U24 103.9 mm to (133.4, 51.7)
- moved U3 96.9 mm to (72.7, 100.8)
- moved D4 93.6 mm to (143.9, 59.6)
- moved J10 93.6 mm to (45.1, 151.2)
- moved RV1 88.1 mm to (119.6, 97.3)
- moved TP1 83.5 mm to (84.3, 107.0)
- moved U14 73.2 mm to (137.6, 115.2)
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
Commit message: Add repo of lib Kicad before analyzing...
Parts:
- added J11: USB_C_Receptacle, CREPP_Connectors_USB:USB_C_Receptacle_GCT_USB4085, F.Cu at (160.2, 155.4)
- added SERVO_SG2: ~, CREPP_Servo:SG90_Servo, F.Cu at (163.1, 122.7)
