File: Kicad_dev/Kicad_dev.kicad_pcb (KiCad board)
At the start: 2 copper layers, 68 parts, among them J1 Conn_01x02_Pin, J10 Screw_Terminal_01x05_2.54mm, J11 USB_C_Receptacle, J2 Conn_01x02_Pin, J3 Conn_01x02_Pin, J4 530470510_Picoblade, J5 Connecteur_SMA, J6 BNC, J7 Screw_Terminal_01x02_2.54mm, J8 Screw_Terminal_01x03_2.54mm, J9 Screw_Terminal_01x04_2.54mm, Q1 IRF540N, Q2 2N7000_THT, Q3 2N7002, SW1 RotaryEncoder_Switch, SW2 RotaryEncoder_Switch, SW3 SW_DPST_x2, SW4 SW_DPST_x2, U1 COM-09032, U11 MAX-8Q, U12 LM317_TO-220, U13 LM7805_TO220, U14 DHT11, U15 DHT11, U17 ATmega328-A, U18 ATmega328-P, U19 STM32F030CCTx, U2 LM317_SOT-223, U20 STM32F446VETx, U21 STM32F723ZETx, U22 MPU-6050, U23 DS1307+, U24 DS3231M, U25 LM358, U26 TP4056, U3 74HC04, U4 L293D, U5 LM358, U6 PC817_SMD, U7 PC817_THT, U8 NEO-M8Q

Commit message: Add repo of lib Kicad before analyzing...
Parts:
- removed SERVO_SG1, SERVO_SG2: ~, CREPP_Servo:SG90_Servo
- added SERVO_SG3: ~, CREPP_Servo:SG90_Servo, F.Cu at (106.6, 120.4)
- added TP2: MM8130-2600, CREPP_Connectors_MURATA:MM8130-2600, F.Cu at (160.8, 111.8)
Connections:
- TP1 pad R: unconnected-(TP1-PadR) -> Net-(TP1-PadR)

Commit message: Add repo of lib Kicad before analyzing...
Parts:
- removed C1: Supercapacitors_D10mm_H20mm, CREPP_Capacitors_THT:C_Radial_D10.0mm_H20.0mm_P5.00mm
- removed SW2: RotaryEncoder_Switch, CREPP_RotaryEncoders:RotaryEncoder
- removed U21: STM32F723ZETx, Package_QFP:LQFP-144_20x20mm_P0.5mm
- added J12: Screw_Terminal_01x05_2.54mm, TerminalBlock_Phoenix:TerminalBlock_Phoenix_MPT-0,5-5-2.54_1x05_P2.54mm_Horizontal, F.Cu at (106.2, 192.0)
- added J13: Screw_Terminal_01x03_2.54mm, TerminalBlock_Phoenix:TerminalBlock_Phoenix_MPT-0,5-3-2.54_1x03_P2.54mm_Horizontal, F.Cu at (132.1, 192.0)
- added J14: Screw_Terminal_01x04_2.54mm, TerminalBlock_Phoenix:TerminalBlock_Phoenix_MPT-0,5-4-2.54_1x04_P2.54mm_Horizontal, F.Cu at (120.4, 192.0)
- added J15: Screw_Terminal_01x02_2.54mm, TerminalBlock_Phoenix:TerminalBlock_Phoenix_MPT-0,5-2-2.54_1x02_P2.54mm_Horizontal, F.Cu at (141.2, 192.0)
- added J16: Screw_Terminal_01x05_2.54mm, TerminalBlock_Phoenix:TerminalBlock_Phoenix_MKDS-1,5-5-5.08_1x05_P5.08mm_Horizontal, F.Cu at (20.3, 190.0)
- added L1: Ferrite_BM, Inductor_SMD:L_0603_1608Metric, F.Cu at (71.6, 166.4)
- added S5: ~, CREPP_Sensors_distance:HC-SR04, F.Cu at (44.2, 91.2)
- added U16: STM32F030CCTx, Package_QFP:LQFP-48_7x7mm_P0.5mm, F.Cu at (36.8, 137.9)
- J10: value Screw_Terminal_01x05_2.54mm -> Screw_Terminal_01x02_2.54mm; footprint TerminalBlock_Phoenix:TerminalBlock_Phoenix_MPT-0,5-5-2.54_1x05_P2.54mm_Horizontal -> TerminalBlock_Phoenix:TerminalBlock_Phoenix_MKDS-1,5-2-5.08_1x02_P5.08mm_Horizontal
- J7: value Screw_Terminal_01x02_2.54mm -> Coon_01x04_Pin_2mm; footprint TerminalBlock_Phoenix:TerminalBlock_Phoenix_MPT-0,5-2-2.54_1x02_P2.54mm_Horizontal -> Connector_JST:JST_PH_B4B-PH-K_1x04_P2.00mm_Vertical
- J8: value Screw_Terminal_01x03_2.54mm -> Screw_Terminal_01x04_2.54mm; footprint TerminalBlock_Phoenix:TerminalBlock_Phoenix_MPT-0,5-3-2.54_1x03_P2.54mm_Horizontal -> TerminalBlock_Phoenix:TerminalBlock_Phoenix_MKDS-1,5-4-5.08_1x04_P5.08mm_Horizontal
- J9: value Screw_Terminal_01x04_2.54mm -> Screw_Terminal_01x03_2.54mm; footprint TerminalBlock_Phoenix:TerminalBlock_Phoenix_MPT-0,5-4-2.54_1x04_P2.54mm_Horizontal -> TerminalBlock_Phoenix:TerminalBlock_Phoenix_MKDS-1,5-3-5.08_1x03_P5.08mm_Horizontal
- U17: value ATmega328-A -> STM32F446VETx; footprint Package_QFP:TQFP-32_7x7mm_P0.8mm -> Package_QFP:LQFP-100_14x14mm_P0.5mm
- U19: value STM32F030CCTx -> STM32F723ZETx; footprint Package_QFP:LQFP-48_7x7mm_P0.5mm -> Package_QFP:LQFP-144_20x20mm_P0.5mm
- U20: value STM32F446VETx -> ATmega328-A; footprint Package_QFP:LQFP-100_14x14mm_P0.5mm -> Package_QFP:TQFP-32_7x7mm_P0.8mm
- moved J8 151.8 mm to (47.2, 190.0)
- moved U17 144.8 mm to (50.3, 160.5), turned to 180 degrees
- moved J11 135.5 mm to (26.5, 133.9), turned to -90 degrees
- moved TP2 133.4 mm to (27.7, 121.1)
- moved SW3 120.9 mm to (98.4, 177.6)
- moved D4 115.1 mm to (92.7, 162.7)
- moved Q2 115.1 mm to (90.6, 168.2)
- moved Q3 115.1 mm to (97.6, 167.4)
- moved J4 112.0 mm to (172.7, 193.6)
- moved U1 110.7 mm to (163.6, 112.0)
- moved J7 110.6 mm to (160.0, 194.3), turned to 180 degrees
- moved SW1 103.8 mm to (156.8, 134.1)
- moved U4 92.0 mm to (149.4, 156.0)
- moved U2 89.6 mm to (104.5, 160.3)
- moved D2 89.6 mm to (102.0, 168.2)
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Connections:
- U17 pad 10: unconnected-(U17-PD6-Pad10) -> Net-(U17-VSS-Pad10)
- U17 pad 21: Net-(U17-GND-Pad21) -> unconnected-(U17-VREF+-Pad21)
- U17 pad 27: unconnected-(U17-PC4-Pad27) -> Net-(U17-VSS-Pad10)
- U17 pad 3: Net-(U17-GND-Pad21) -> unconnected-(U17-PE4-Pad3)
- U17 pad 4: Net-(U17-VCC-Pad4) -> unconnected-(U17-PE5-Pad4)
- U17 pad 5: Net-(U17-GND-Pad21) -> unconnected-(U17-PE6-Pad5)
- U17 pad 6: Net-(U17-VCC-Pad4) -> unconnected-(U17-VBAT-Pad6)
- U19 pad 16: unconnected-(U19-PA6-Pad16) -> Net-(U19-VSS-Pad107)
- U19 pad 23: Net-(U19-VSS-Pad23) -> unconnected-(U19-PH0-Pad23)
- U19 pad 35: Net-(U19-VSS-Pad23) -> unconnected-(U19-PA1-Pad35)
- U19 pad 38: unconnected-(U19-PA15-Pad38) -> Net-(U19-VSS-Pad107)
- U19 pad 47: Net-(U19-VSS-Pad23) -> unconnected-(U19-PB1-Pad47)
- U20 pad 10: Net-(U20-VSS-Pad10) -> unconnected-(U20-PD6-Pad10)
- U20 pad 21: unconnected-(U20-VREF+-Pad21) -> Net-(U20-GND-Pad21)
- U20 pad 27: Net-(U20-VSS-Pad10) -> unconnected-(U20-PC4-Pad27)
- U20 pad 3: unconnected-(U20-PE4-Pad3) -> Net-(U20-GND-Pad21)
- U20 pad 4: unconnected-(U20-PE5-Pad4) -> Net-(U20-VCC-Pad4)
- U20 pad 5: unconnected-(U20-PE6-Pad5) -> Net-(U20-GND-Pad21)
- U20 pad 6: unconnected-(U20-VBAT-Pad6) -> Net-(U20-VCC-Pad4)

Commit message: Add OLED PCB mount
Parts:
- added RV1: R_Potentiometer, Potentiometer_THT:Potentiometer_Alps_RK163_Single_Horizontal, F.Cu at (208.4, 131.3)
- added S5: ~, CREPP_Sensors_distance:HC-SR04, F.Cu at (216.6, 133.7)
- added U1: MPU-6050, Sensor_Motion:InvenSense_QFN-24_4x4mm_P0.5mm, F.Cu at (180.1, 153.2)
- added U21: COM-09032, CREPP_Joysticks_SW:XDCR_COM-09032, F.Cu at (202.9, 112.6)
- U8: value NEO-M8Q -> NEO-M8Q

Commit message: Add OLED PCB mount
Parts:
- removed the RV1 at (208.4, 131.3)
- removed U21: COM-09032, CREPP_Joysticks_SW:XDCR_COM-09032
- added OLED_1: ~, CREPP_Screens:SSD1306_OLED_0.96_PCB, F.Cu at (131.5, 59.4)
- S1: footprint CREPP_Spacers:Spacer_M3_FF_05mm -> CREPP_Spacers:Spacer_M3_MF_05mm
- S2: footprint CREPP_Spacers:Spacer_M3_FF_10mm -> CREPP_Spacers:Spacer_M3_MF_05mm
- S3: footprint CREPP_Spacers:Spacer_M3_FF_15mm -> CREPP_Spacers:Spacer_M3_MF_05mm
- S4: footprint CREPP_Spacers:Spacer_M3_FF_20mm -> CREPP_Spacers:Spacer_M3_MF_05mm
- moved S5 64.6 mm to (178.5, 81.5)

Commit message: Update
Parts:
- removed the U1 at (163.6, 112.0)
- added U21: COM-09032, CREPP_Joysticks_SW:XDCR_COM-09032, F.Cu at (165.4, 108.8)
- moved OLED1 101.5 mm to (227.0, 93.0)
- moved OLED_1 73.8 mm to (197.0, 93.4)
- moved RV1 7.23 mm to (101.5, 86.0), turned to -90 degrees

Commit message: Update
Parts:
- removed U22: MPU-6050, Sensor_Motion:InvenSense_QFN-24_4x4mm_P0.5mm
