File: Kicad_dev/Modules/Sensors.kicad_sch (KiCad schematic)
At the start: 4 parts, among them U1 MPU-6050, U21 COM-09032

Commit message: Update
Parts:
- RV1: footprint Potentiometer_THT:Potentiometer_Alps_RK163_Single_Horizontal -> CREPP_Potentiometers:Potentiometer_Alps_RK09Y11_Single_Horizontal
Changed lines of the file:
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@@
 	(symbol
 		(lib_id "CREPP_Potentiometers_THT:R_Potentiometer")
-		(at 240.03 90.17 0)
+		(at 152.4 110.49 0)
 		(unit 1)
 		(exclude_from_sim no)
@@
 		(fields_autoplaced yes)
 		(property "Reference" "RV1"
-			(at 237.49 88.8999 0)
+			(at 149.86 109.2199 0)
 			(effects
 				(font
@@
 		)
 		(property "Value" "R_Potentiometer"
-			(at 237.49 91.4399 0)
+			(at 149.86 111.7599 0)
 			(effects
 				(font
@@
 			)
 		)
-		(property "Footprint" "Potentiometer_THT:Potentiometer_Alps_RK163_Single_Horizontal"
-			(at 240.03 90.17 0)
+		(property "Footprint" "CREPP_Potentiometers:Potentiometer_Alps_RK09Y11_Single_Horizontal"
+			(at 152.4 110.49 0)
 			(effects
 				(font
@@
 		)
 		(property "Datasheet" "~"
-			(at 240.03 90.17 0)
+			(at 152.4 110.49 0)
 			(effects
 				(font
@@
 		)
 		(property "Description" "Potentiometer"
-			(at 240.03 90.17 0)
+			(at 152.4 110.49 0)
 			(effects
 				(font
@@
 			)
 		)
-		(pin "2"
+		(pin "3"
 		)
 		(pin "1"
 		)
-		(pin "3"
+		(pin "2"
 		)
 		(instances
-			(project "Kicad_dev"
+			(project ""
 				(path "/8104dfe2-da9a-40cd-b518-c622bfb26061/7c3c07de-3c76-4af0-8fc4-525102bf82ab"
 					(reference "RV1")
