File: Kicad_dev/Modules/Signals.kicad_sch (KiCad schematic)
At the start: 2 parts, among them U30 NRF24L01_Breakout [CREPP]

Commit message: Update
Parts:
- removed U30: NRF24L01_Breakout [CREPP], CREPP_NRF24:nRF24L01_Breakout, symbol CREPP_NRF24:NRF24L01_Breakout
- added U22: NRF24L01_Breakout, CREPP_NRF24:nRF24L01_Breakout, symbol CREPP_NRF24:NRF24L01_Breakout
- added U28: ~, symbol CREPP_NRF24:NRF24_Virtual
Changed lines of the file:
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@@
 	(paper "A4")
+	(symbol
+		(lib_id "CREPP_NRF24:NRF24L01_Breakout ")
+		(at 189.23 90.17 0)
+		(unit 1)
+		(exclude_from_sim no)
+		(in_bom yes)
+		(on_board yes)
+		(dnp no)
+		(fields_autoplaced yes)
+		(property "Reference" "U22"
+			(at 199.39 88.8999 0)
+			(effects
+				(font
+					(size 1.27 1.27)
+				)
+				(justify left)
+			)
+		)
+		(property "Value" "NRF24L01_Breakout"
+			(at 199.39 91.4399 0)
+			(effects
+				(font
+					(size 1.27 1.27)
+				)
+				(justify left)
+			)
+		)
+		(property "Footprint" "CREPP_NRF24:nRF24L01_Breakout"
+			(at 193.04 74.93 0)
+			(effects
+				(font
+					(size 1.27 1.27)
+					(italic yes)
+				)
+				(justify left)
+				(hide yes)
+			)
+		)
+		(property "Datasheet" "http://www.nordicsemi.com/eng/content/download/2730/34105/file/nRF24L01_Product_Specification_v2_0.pdf"
+			(at 189.23 92.71 0)
+			(effects
+				(font
+					(size 1.27 1.27)
+				)
+				(hide yes)
+			)
+		)
+		(property "Description" "Ultra low power 2.4GHz RF Transceiver, Carrier PCB"
+			(at 189.23 90.17 0)
+			(effects
+				(font
+					(size 1.27 1.27)
+				)
+				(hide yes)
+			)
+		)
+		(pin "1"
+		)
+		(pin "2"
+		)
+		(pin "8"
+		)
+		(pin "5"
+		)
+		(pin "3"
+		)
+		(pin "6"
+		)
+		(pin "7"
+		)
+		(pin "4"
+		)
+		(instances
+			(project ""
+				(path "/8104dfe2-da9a-40cd-b518-c622bfb26061/1034155c-8abf-469a-b01c-35ece3b3f3d3"
+					(reference "U22")
+					(unit 1)
+				)
+			)
+		)
+	)
+	(symbol
+		(lib_id "CREPP_NRF24:NRF24_Virtual")
+		(at 148.59 110.49 0)
+		(unit 1)
+		(exclude_from_sim no)
+		(in_bom yes)
+		(on_board yes)
+		(dnp no)
+		(fields_autoplaced yes)
+		(property "Reference" "U28"
+			(at 154.94 105.4099 0)
+			(effects
+				(font
+					(size 1.27 1.27)
+				)
+				(justify left)
+			)
+		)
+		(property "Value" "~"
+			(at 154.94 107.315 0)
+			(effects
+				(font
+					(size 1.27 1.27)
+				)
+				(justify left)
+			)
+		)
+		(property "Footprint" ""
+			(at 148.59 110.49 0)
+			(effects
+				(font
+					(size 1.27 1.27)
+				)
+				(hide yes)
+			)
+		)
+		(property "Datasheet" ""
+			(at 148.59 110.49 0)
+			(effects
+				(font
+					(size 1.27 1.27)
+				)
+				(hide yes)
+			)
+		)
+		(property "Description" ""
+			(at 148.59 110.49 0)
+			(effects
+				(font
+					(size 1.27 1.27)
+				)
+				(hide yes)
+			)
+		)
+		(instances
+			(project ""
+				(path "/8104dfe2-da9a-40cd-b518-c622bfb26061/1034155c-8abf-469a-b01c-35ece3b3f3d3"
+					(reference "U28")
+					(unit 1)
+				)
+			)
+		)
+	)
 	(symbol
 		(lib_id "CREPP_Bluetooth:Bluetooth HC-05 [CREPP_VIRTUAL]")
@@
 					(unit 1)
 				)
-			)
-		)
-	)
-	(symbol
-		(lib_id "CREPP_NRF24:NRF24L01_Breakout ")
-		(at 110.49 125.73 0)
-		(unit 1)
-		(exclude_from_sim no)
-		(in_bom yes)
-		(on_board yes)
-		(dnp no)
-		(fields_autoplaced yes)
-		(property "Reference" "U30"
-			(at 120.65 124.4599 0)
-			(effects
-				(font
-					(size 1.27 1.27)
-				)
-				(justify left)
-			)
-		)
-		(property "Value" "NRF24L01_Breakout [CREPP]"
-			(at 120.65 126.9999 0)
-			(effects
-				(font
-					(size 1.27 1.27)
-				)
-				(justify left)
-			)
-		)
-		(property "Footprint" "CREPP_NRF24:nRF24L01_Breakout"
-			(at 114.3 110.49 0)
-			(effects
-				(font
-					(size 1.27 1.27)
-					(italic yes)
-				)
-				(justify left)
-				(hide yes)
-			)
-		)
-		(property "Datasheet" "http://www.nordicsemi.com/eng/content/download/2730/34105/file/nRF24L01_Product_Specification_v2_0.pdf"
-			(at 110.49 128.27 0)
-			(effects
-				(font
-					(size 1.27 1.27)
-				)
-				(hide yes)
-			)
-		)
-		(property "Description" "Ultra low power 2.4GHz RF Transceiver, Carrier PCB"
-			(at 110.49 125.73 0)
-			(effects
-				(font
-					(size 1.27 1.27)
-				)
-				(hide yes)
-			)
-		)
-		(pin "8"
-		)
-		(pin "3"
-		)
-		(pin "2"
-		)
-		(pin "1"
-		)
-		(pin "7"
-		)
-		(pin "4"
-		)
-		(pin "5"
-		)
-		(pin "6"
-		)
-		(instances
-			(project ""
-				(path "/8104dfe2-da9a-40cd-b518-c622bfb26061/1034155c-8abf-469a-b01c-35ece3b3f3d3"
-					(reference "U30")
-					(unit 1)
-				)

Commit message: Update
Parts:
- removed U22: NRF24L01_Breakout, CREPP_NRF24:nRF24L01_Breakout, symbol CREPP_NRF24:NRF24L01_Breakout
- added U22: NRF24L01_Breakout_socket, CREPP_NRF24:nRF24L01_Breakout, symbol CREPP_NRF24:NRF24L01_Breakout _Socket
Changed lines of the file:
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@@
 	(paper "A4")
 	(symbol
-		(lib_id "CREPP_NRF24:NRF24L01_Breakout ")
-		(at 189.23 90.17 0)
+		(lib_id "CREPP_NRF24:NRF24L01_Breakout _Socket")
+		(at 187.96 111.76 0)
 		(unit 1)
 		(exclude_from_sim no)
@@
 		(fields_autoplaced yes)
 		(property "Reference" "U22"
-			(at 199.39 88.8999 0)
+			(at 198.12 110.4899 0)
 			(effects
 				(font
@@
 			)
 		)
-		(property "Value" "NRF24L01_Breakout"
-			(at 199.39 91.4399 0)
+		(property "Value" "NRF24L01_Breakout_socket"
+			(at 198.12 113.0299 0)
 			(effects
 				(font
@@
 		)
 		(property "Footprint" "CREPP_NRF24:nRF24L01_Breakout"
-			(at 193.04 74.93 0)
+			(at 191.77 96.52 0)
 			(effects
 				(font
@@
 		)
 		(property "Datasheet" "http://www.nordicsemi.com/eng/content/download/2730/34105/file/nRF24L01_Product_Specification_v2_0.pdf"
-			(at 189.23 92.71 0)
+			(at 187.96 114.3 0)
 			(effects
 				(font
@@
 		)
 		(property "Description" "Ultra low power 2.4GHz RF Transceiver, Carrier PCB"
-			(at 189.23 90.17 0)
+			(at 187.96 111.76 0)
 			(effects
 				(font
@@
 		(pin "1"
 		)
+		(pin "5"
+		)
+		(pin "6"
+		)
+		(pin "4"
+		)
 		(pin "2"
 		)
 		(pin "8"
 		)
-		(pin "5"
+		(pin "7"
 		)
 		(pin "3"
 		)
-		(pin "6"
-		)
-		(pin "7"
-		)
-		(pin "4"
-		)
 		(instances
